File: preamplifier/preamplifier.sch (KiCad schematic (older format))
At the start: 0 parts

Commit message: LOL
Parts:
- added C?: 1000p, symbol Device:C
- added C? (x3): 2.2u, symbol Device:C
- added J? (x2): Conn_01x02_Female, symbol Connector:Conn_01x02_Female
- added R? (x2): 2k, symbol Device:R
- added R? (x2): 10k, symbol Device:R
- added R? (x3): 100k, symbol Device:R
- added R?: 50, symbol Device:R
- added RV?: 50k, symbol Device:R_POT
- added RV?: 200k, symbol Device:R_POT
- added U? (x3): OPA1678, symbol Amplifier_Operational:OPA1678
Connections:
- new net: C?.1, R?.1, R?.2, U?.1
- new net: C?.1, C?.2, RV?.1, U?.2 (-)
- new net: C?.1, R?.1, R?.2, U?.3 (+)
- new net: R?.1, R?.2, U?.5 (+)
- new net: U?.6 (-), U?.7
- new net: R?.2, RV?.2
- new net: C?.2, J?.2 (Pin_2), RV?.2
- new net: R?.2, RV?.1
- new net: C?.2, R?.1
- new net: C?.1, J?.1 (Pin_1), R?.2
- new net GND: C?.2, J?.1 (Pin_1), J?.2 (Pin_2), R?.1, R?.2, R?.2, U?.4 (V-)
- new net VCC: R?.1, R?.1, R?.1, U?.8 (V+)
