File: MatrixDriver/MatrixDriver.sch (KiCad schematic (older format))
At the start: 391 parts

Commit message: Laptop Push
Parts:
- removed D? (x39): LED, symbol Device:LED
- added R1, R10, R11, R12, R13, R14, R15, R16, R17, R18, R19, R2, R20, R21, R22, R23, R24, R25, R26, R27, R28, R29, R3, R30, R31, R32, R33, R34, R35, R36, R37, R38, R39, R4, R5, R6, R7, R8, R9: R, symbol Device:R
- gave numbers to parts that had none: 352
Connections:
- net at U1.1 (CS34): now also R6.2
- net at U1.10 (SW8): now also D40.2 (A), D41.2 (A), D42.2 (A), D43.2 (A), D44.2 (A), D45.2 (A), D46.2 (A), D47.2 (A), D48.2 (A), D49.2 (A), D50.2 (A), D51.2 (A), D52.2 (A), D53.2 (A), D54.2 (A), D55.2 (A), D56.2 (A), D57.2 (A), D58.2 (A), D59.2 (A), D60.2 (A), D61.2 (A), D62.2 (A), D63.2 (A), D64.2 (A), D65.2 (A), D66.2 (A), D67.2 (A), D68.2 (A), D69.2 (A), D70.2 (A), D71.2 (A), D72.2 (A), D73.2 (A), D74.2 (A), D75.2 (A), D76.2 (A), D77.2 (A), D78.2 (A)
- net at U1.11 (SW9): now also D1.2 (A), D10.2 (A), D11.2 (A), D12.2 (A), D13.2 (A), D14.2 (A), D15.2 (A), D16.2 (A), D17.2 (A), D18.2 (A), D19.2 (A), D2.2 (A), D20.2 (A), D21.2 (A), D22.2 (A), D23.2 (A), D24.2 (A), D25.2 (A), D26.2 (A), D27.2 (A), D28.2 (A), D29.2 (A), D3.2 (A), D30.2 (A), D31.2 (A), D32.2 (A), D33.2 (A), D34.2 (A), D35.2 (A), D36.2 (A), D37.2 (A), D38.2 (A), D39.2 (A), D4.2 (A), D5.2 (A), D6.2 (A), D7.2 (A), D8.2 (A), D9.2 (A)
- net at U1.2 (SW1): now also R5.2
- net at U1.26 (CS1): now also R39.2
- net at U1.27 (CS2): now also R38.2
- net at U1.28 (CS3): now also R37.2
- net at U1.29 (CS4): now also R36.2
- net at U1.3 (SW2): now also R4.2
- net at U1.30 (CS5): now also R35.2
- net at U1.31 (CS6): now also R34.2
- net at U1.32 (CS7): now also R33.2
- net at U1.33 (CS8): now also R32.2
- net at U1.34 (CS9): now also R31.2
- net at U1.35 (CS10): now also R30.2
- net at U1.37 (CS11): now also R29.2
- net at U1.38 (CS12): now also R28.2
- net at U1.39 (CS13): now also R27.2
- net at U1.4 (SW3): now also R3.2
- net at U1.40 (CS14): now also R26.2
- net at U1.41 (CS15): now also R25.2
- net at U1.42 (CS16): now also R24.2
- net at U1.43 (CS17): now also R23.2
- net at U1.44 (CS18): now also R22.2
- net at U1.45 (CS19): now also R21.2
- net at U1.46 (CS20): now also R20.2
- net at U1.47 (CS21): now also R19.2
- net at U1.48 (CS22): now also R18.2
- net at U1.49 (CS23): now also R17.2
- net at U1.5 (CS38): now also R2.2
- net at U1.50 (CS24): now also R16.2
- net at U1.51 (CS25): now also R15.2
- net at U1.52 (CS26): now also R14.2
- net at U1.53 (CS27): now also R13.2
- net at U1.54 (CS28): now also R12.2
- net at U1.56 (CS29): now also R11.2
- net at U1.57 (CS30): now also R10.2
- net at U1.58 (CS31): now also R9.2
- net at U1.59 (CS32): now also R8.2
- net at U1.6 (SW4): now also R1.2
- net at U1.60 (CS33): now also R7.2
- net at U1.7 (SW5): now also D157.2 (A), D158.2 (A), D159.2 (A), D160.2 (A), D161.2 (A), D162.2 (A), D163.2 (A), D164.2 (A), D165.2 (A), D166.2 (A), D167.2 (A), D168.2 (A), D169.2 (A), D170.2 (A), D171.2 (A), D172.2 (A), D173.2 (A), D174.2 (A), D175.2 (A), D176.2 (A), D177.2 (A), D178.2 (A), D179.2 (A), D180.2 (A), D181.2 (A), D182.2 (A), D183.2 (A), D184.2 (A), D185.2 (A), D186.2 (A), D187.2 (A), D188.2 (A), D189.2 (A), D190.2 (A), D191.2 (A), D192.2 (A), D193.2 (A), D194.2 (A), D195.2 (A)
- net at U1.8 (SW6): now also D118.2 (A), D119.2 (A), D120.2 (A), D121.2 (A), D122.2 (A), D123.2 (A), D124.2 (A), D125.2 (A), D126.2 (A), D127.2 (A), D128.2 (A), D129.2 (A), D130.2 (A), D131.2 (A), D132.2 (A), D133.2 (A), D134.2 (A), D135.2 (A), D136.2 (A), D137.2 (A), D138.2 (A), D139.2 (A), D140.2 (A), D141.2 (A), D142.2 (A), D143.2 (A), D144.2 (A), D145.2 (A), D146.2 (A), D147.2 (A), D148.2 (A), D149.2 (A), D150.2 (A), D151.2 (A), D152.2 (A), D153.2 (A), D154.2 (A), D155.2 (A), D156.2 (A)
- net at U1.9 (SW7): now also D100.2 (A), D101.2 (A), D102.2 (A), D103.2 (A), D104.2 (A), D105.2 (A), D106.2 (A), D107.2 (A), D108.2 (A), D109.2 (A), D110.2 (A), D111.2 (A), D112.2 (A), D113.2 (A), D114.2 (A), D115.2 (A), D116.2 (A), D117.2 (A), D79.2 (A), D80.2 (A), D81.2 (A), D82.2 (A), D83.2 (A), D84.2 (A), D85.2 (A), D86.2 (A), D87.2 (A), D88.2 (A), D89.2 (A), D90.2 (A), D91.2 (A), D92.2 (A), D93.2 (A), D94.2 (A), D95.2 (A), D96.2 (A), D97.2 (A), D98.2 (A), D99.2 (A)
- net at D117.1 (K): now also D156.1 (K), D195.1 (K), D234.1 (K), D273.1 (K), D312.1 (K), D351.1 (K), D39.1 (K), D78.1 (K), R1.1
- net at D116.1 (K): now also D155.1 (K), D194.1 (K), D233.1 (K), D272.1 (K), D311.1 (K), D350.1 (K), D38.1 (K), D77.1 (K), R2.1
- net at D115.1 (K): now also D154.1 (K), D193.1 (K), D232.1 (K), D271.1 (K), D310.1 (K), D349.1 (K), D37.1 (K), D76.1 (K), R3.1
- net at D114.1 (K): now also D153.1 (K), D192.1 (K), D231.1 (K), D270.1 (K), D309.1 (K), D348.1 (K), D36.1 (K), D75.1 (K), R4.1
- net at D113.1 (K): now also D152.1 (K), D191.1 (K), D230.1 (K), D269.1 (K), D308.1 (K), D347.1 (K), D35.1 (K), D74.1 (K), R5.1
- net at D112.1 (K): now also D151.1 (K), D190.1 (K), D229.1 (K), D268.1 (K), D307.1 (K), D34.1 (K), D346.1 (K), D73.1 (K), R6.1
- net at D111.1 (K): now also D150.1 (K), D189.1 (K), D228.1 (K), D267.1 (K), D306.1 (K), D33.1 (K), D345.1 (K), D72.1 (K), R7.1
- net at D110.1 (K): now also D149.1 (K), D188.1 (K), D227.1 (K), D266.1 (K), D305.1 (K), D32.1 (K), D344.1 (K), D71.1 (K), R8.1
- net at D109.1 (K): now also D148.1 (K), D187.1 (K), D226.1 (K), D265.1 (K), D304.1 (K), D31.1 (K), D343.1 (K), D70.1 (K), R9.1
- net at D108.1 (K): now also D147.1 (K), D186.1 (K), D225.1 (K), D264.1 (K), D30.1 (K), D303.1 (K), D342.1 (K), D69.1 (K), R10.1
- net at D107.1 (K): now also D146.1 (K), D185.1 (K), D224.1 (K), D263.1 (K), D29.1 (K), D302.1 (K), D341.1 (K), D68.1 (K), R11.1
- net at D106.1 (K): now also D145.1 (K), D184.1 (K), D223.1 (K), D262.1 (K), D28.1 (K), D301.1 (K), D340.1 (K), D67.1 (K), R12.1
- net at D105.1 (K): now also D144.1 (K), D183.1 (K), D222.1 (K), D261.1 (K), D27.1 (K), D300.1 (K), D339.1 (K), D66.1 (K), R13.1
- net at D104.1 (K): now also D143.1 (K), D182.1 (K), D221.1 (K), D26.1 (K), D260.1 (K), D299.1 (K), D338.1 (K), D65.1 (K), R14.1
- net at D103.1 (K): now also D142.1 (K), D181.1 (K), D220.1 (K), D25.1 (K), D259.1 (K), D298.1 (K), D337.1 (K), D64.1 (K), R15.1
- net at D102.1 (K): now also D141.1 (K), D180.1 (K), D219.1 (K), D24.1 (K), D258.1 (K), D297.1 (K), D336.1 (K), D63.1 (K), R16.1
- net at D101.1 (K): now also D140.1 (K), D179.1 (K), D218.1 (K), D23.1 (K), D257.1 (K), D296.1 (K), D335.1 (K), D62.1 (K), R17.1
- net at D100.1 (K): now also D139.1 (K), D178.1 (K), D217.1 (K), D22.1 (K), D256.1 (K), D295.1 (K), D334.1 (K), D61.1 (K), R18.1
- net at D99.1 (K): now also D138.1 (K), D177.1 (K), D21.1 (K), D216.1 (K), D255.1 (K), D294.1 (K), D333.1 (K), D60.1 (K), R19.1
- net at D98.1 (K): now also D137.1 (K), D176.1 (K), D20.1 (K), D215.1 (K), D254.1 (K), D293.1 (K), D332.1 (K), D59.1 (K), R20.1
- net at D97.1 (K): now also D136.1 (K), D175.1 (K), D19.1 (K), D214.1 (K), D253.1 (K), D292.1 (K), D331.1 (K), D58.1 (K), R21.1
- net at D96.1 (K): now also D135.1 (K), D174.1 (K), D18.1 (K), D213.1 (K), D252.1 (K), D291.1 (K), D330.1 (K), D57.1 (K), R22.1
- net at D95.1 (K): now also D134.1 (K), D17.1 (K), D173.1 (K), D212.1 (K), D251.1 (K), D290.1 (K), D329.1 (K), D56.1 (K), R23.1
- net at D94.1 (K): now also D133.1 (K), D16.1 (K), D172.1 (K), D211.1 (K), D250.1 (K), D289.1 (K), D328.1 (K), D55.1 (K), R24.1
- net at D93.1 (K): now also D132.1 (K), D15.1 (K), D171.1 (K), D210.1 (K), D249.1 (K), D288.1 (K), D327.1 (K), D54.1 (K), R25.1
- net at D92.1 (K): now also D131.1 (K), D14.1 (K), D170.1 (K), D209.1 (K), D248.1 (K), D287.1 (K), D326.1 (K), D53.1 (K), R26.1
- net at D91.1 (K): now also D13.1 (K), D130.1 (K), D169.1 (K), D208.1 (K), D247.1 (K), D286.1 (K), D325.1 (K), D52.1 (K), R27.1
- net at D90.1 (K): now also D12.1 (K), D129.1 (K), D168.1 (K), D207.1 (K), D246.1 (K), D285.1 (K), D324.1 (K), D51.1 (K), R28.1
- net at D89.1 (K): now also D11.1 (K), D128.1 (K), D167.1 (K), D206.1 (K), D245.1 (K), D284.1 (K), D323.1 (K), D50.1 (K), R29.1
- net at D88.1 (K): now also D10.1 (K), D127.1 (K), D166.1 (K), D205.1 (K), D244.1 (K), D283.1 (K), D322.1 (K), D49.1 (K), R30.1
- net at D87.1 (K): now also D126.1 (K), D165.1 (K), D204.1 (K), D243.1 (K), D282.1 (K), D321.1 (K), D48.1 (K), D9.1 (K), R31.1
- net at D86.1 (K): now also D125.1 (K), D164.1 (K), D203.1 (K), D242.1 (K), D281.1 (K), D320.1 (K), D47.1 (K), D8.1 (K), R32.1
- net at D85.1 (K): now also D124.1 (K), D163.1 (K), D202.1 (K), D241.1 (K), D280.1 (K), D319.1 (K), D46.1 (K), D7.1 (K), R33.1
- net at D84.1 (K): now also D123.1 (K), D162.1 (K), D201.1 (K), D240.1 (K), D279.1 (K), D318.1 (K), D45.1 (K), D6.1 (K), R34.1
- net at D83.1 (K): now also D122.1 (K), D161.1 (K), D200.1 (K), D239.1 (K), D278.1 (K), D317.1 (K), D44.1 (K), D5.1 (K), R35.1
- net at D82.1 (K): now also D121.1 (K), D160.1 (K), D199.1 (K), D238.1 (K), D277.1 (K), D316.1 (K), D4.1 (K), D43.1 (K), R36.1
- net at D81.1 (K): now also D120.1 (K), D159.1 (K), D198.1 (K), D237.1 (K), D276.1 (K), D3.1 (K), D315.1 (K), D42.1 (K), R37.1
- net at D80.1 (K): now also D119.1 (K), D158.1 (K), D197.1 (K), D2.1 (K), D236.1 (K), D275.1 (K), D314.1 (K), D41.1 (K), R38.1
- net at D79.1 (K): now also D1.1 (K), D118.1 (K), D157.1 (K), D196.1 (K), D235.1 (K), D274.1 (K), D313.1 (K), D40.1 (K), R39.1
- net at D196.2 (A), D197.2 (A), D198.2 (A)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: now also U1.6 (SW4)
- net at D235.2 (A), D236.2 (A), D237.2 (A)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: now also U1.4 (SW3)
- net at D274.2 (A), D275.2 (A), D276.2 (A)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: now also U1.3 (SW2)
- net at D313.2 (A), D314.2 (A), D315.2 (A)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: now also U1.2 (SW1)
Other:
- moved on the sheet: D1, D10, D100, D101, D102, D103, D104, D105, D106, D107, D108, D109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
