File: MotorcycleSwitch - Rev2/MotorcycleSwitch.sch (KiCad schematic (older format))
At the start: 66 parts, among them J1 AdafruitConverter, J2 Conn_01x07_Female, Q4 Q_DUAL_NMOS_PMOS_BSD235CH6327, SW1 SW_Push, SW2 SW_Push, SW3 SW_Push, SW4 SW_Push, SW5 SW_Push, U1 TPS4H160-A, U2 STM32G030C6T6, U3 BD433M2WEFJ-CE2

Commit message: Laptop Push
Parts:
- R14, R20, R22, R23, R24: value 510 -> 250
- R15, R16, R17, R18, R19: value 200 -> 100
Other:
- note added: "(3.3V-2.9V)/100ohm = 4mA"
- note removed: "(3.3V-3.2V)/20ohm = 5mA"
Changed lines of the file:
@@
 P 850 9700
 F 0 "R15" H 920 9746 50  0000 L CNN
-F 1 "200" H 920 9655 50  0000 L CNN
+F 1 "100" H 920 9655 50  0000 L CNN
 F 2 "Resistor_SMD:R_0603_1608Metric" V 780 9700 50  0001 C CNN
 F 3 "~" H 850 9700 50  0001 C CNN
@@
 P 1100 9700
 F 0 "R16" H 1170 9746 50  0000 L CNN
-F 1 "200" H 1170 9655 50  0000 L CNN
+F 1 "100" H 1170 9655 50  0000 L CNN
 F 2 "Resistor_SMD:R_0603_1608Metric" V 1030 9700 50  0001 C CNN
 F 3 "~" H 1100 9700 50  0001 C CNN
@@
 P 1350 9700
 F 0 "R17" H 1420 9746 50  0000 L CNN
-F 1 "200" H 1420 9655 50  0000 L CNN
+F 1 "100" H 1420 9655 50  0000 L CNN
 F 2 "Resistor_SMD:R_0603_1608Metric" V 1280 9700 50  0001 C CNN
 F 3 "~" H 1350 9700 50  0001 C CNN
@@
 P 1600 9700
 F 0 "R18" H 1670 9746 50  0000 L CNN
-F 1 "200" H 1670 9655 50  0000 L CNN
+F 1 "100" H 1670 9655 50  0000 L CNN
 F 2 "Resistor_SMD:R_0603_1608Metric" V 1530 9700 50  0001 C CNN
 F 3 "~" H 1600 9700 50  0001 C CNN
@@
 P 1850 9700
 F 0 "R19" H 1920 9746 50  0000 L CNN
-F 1 "200" H 1920 9655 50  0000 L CNN
+F 1 "100" H 1920 9655 50  0000 L CNN
 F 2 "Resistor_SMD:R_0603_1608Metric" V 1780 9700 50  0001 C CNN
 F 3 "~" H 1850 9700 50  0001 C CNN
@@
 PA_PTT_N
 Text Notes 700  7800 0    50   ~ 0
-(3.3V-3.2V)/20ohm = 5mA
+(3.3V-2.9V)/100ohm = 4mA
 Wire Wire Line
 	12000 6000 11650 6000
@@
 P 2650 9700
 F 0 "R14" H 2720 9746 50  0000 L CNN
-F 1 "510" H 2720 9655 50  0000 L CNN
+F 1 "250" H 2720 9655 50  0000 L CNN
 F 2 "Resistor_SMD:R_0603_1608Metric" V 2580 9700 50  0001 C CNN
 F 3 "~" H 2650 9700 50  0001 C CNN
@@
 P 2900 9700
 F 0 "R20" H 2970 9746 50  0000 L CNN
-F 1 "510" H 2970 9655 50  0000 L CNN
+F 1 "250" H 2970 9655 50  0000 L CNN
 F 2 "Resistor_SMD:R_0603_1608Metric" V 2830 9700 50  0001 C CNN
 F 3 "~" H 2900 9700 50  0001 C CNN
@@
 P 3400 9700
 F 0 "R23" H 3470 9746 50  0000 L CNN
-F 1 "510" H 3470 9655 50  0000 L CNN
+F 1 "250" H 3470 9655 50  0000 L CNN
 F 2 "Resistor_SMD:R_0603_1608Metric" V 3330 9700 50  0001 C CNN
 F 3 "~" H 3400 9700 50  0001 C CNN
@@
 P 3650 9700
 F 0 "R24" H 3720 9746 50  0000 L CNN
-F 1 "510" H 3720 9655 50  0000 L CNN
+F 1 "250" H 3720 9655 50  0000 L CNN
 F 2 "Resistor_SMD:R_0603_1608Metric" V 3580 9700 50  0001 C CNN
 F 3 "~" H 3650 9700 50  0001 C CNN
@@
 P 3150 9700
 F 0 "R22" H 3220 9746 50  0000 L CNN
-F 1 "510" H 3220 9655 50  0000 L CNN
+F 1 "250" H 3220 9655 50  0000 L CNN
 F 2 "Resistor_SMD:R_0603_1608Metric" V 3080 9700 50  0001 C CNN
 F 3 "~" H 3150 9700 50  0001 C CNN

Commit message: Laptop Push
Parts:
- R2: value 650 -> 1k
- R21: value 100 -> 200
Other:
- note added: "For current limiting in case of \naccidental shoot through"
- note added: "For version A, four individual STx pins report the fault conditions, each pin for its \nrespective channel. When a fault condition occurs, it pulls STx down to GND.A 3.3- or 5-V \nexternalpullup is required to match the supply level of the \nmicrocontroller.The digital status of each channel can be reported individually,or \nglobally by connecting all the STx pins together"
- note added: "Rcl = [0.8 * 2500] / Iout(A)\nRcl = [0.8 * 2500] / 2A(limit) = 1kohm"
- note added: "The DIAG_EN pin enables or disables the diagnostic functions.\nIf multiple devices are used,but the ADCresourceis limited in \nthe microcontroller,the MCU can use GPIOs to set DIAG_EN high to\n enable the diagnostics of one device while disabling the \ndiagnostics of the other devices by setting DIAG_EN low. In addition,\nthe device can keep the power consumption to a minimum by \nsetting DIAG_EN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"
- note removed: "Add 2x5 prog header"
- note removed: "For version A, four individual STx pins report the fault conditions, each pin for its \nrespective channel. When a fault condition occurs, it pulls STx down to GND.A 3.3- or 5-V \nexternalpullup is requiredto match the supply level of the \nmicrocontroller.The digital status of each channel can be reported individually,or \nglobally by connecting all the STx pins together"
- note removed: "Rcl = [0.8V * 2500] / Iout(A)"
- note removed: "\n\n Determine quiescent current of rev1 - change rev2 if needed\n Include diagnostic feedback from load driver to red LED's (user)\n Include robust software debouncing\nFix Schotky\n\n"
- moved on the sheet: J1
Changed lines of the file:
@@
 Wire Wire Line
 	11400 6750 11400 7150
-Text Notes 11100 4750 0    50   ~ 0
-For version A, four individual STx pins report the fault conditions, each pin for its \nrespective channel. When a fault condition occurs, it pulls STx down to GND.A 3.3- or 5-V \nexternalpullup is requiredto match the supply level of the \nmicrocontroller.The digital status of each channel can be reported individually,or \nglobally by connecting all the STx pins together
+Text Notes 11100 3925 0    50   ~ 0
+For version A, four individual STx pins report the fault conditions, each pin for its \nrespective channel. When a fault condition occurs, it pulls STx down to GND.A 3.3- or 5-V \nexternalpullup is required to match the supply level of the \nmicrocontroller.The digital status of each channel can be reported individually,or \nglobally by connecting all the STx pins together
 $Comp
 L Device:R R2
@@
 P 11150 6900
 F 0 "R2" H 11220 6946 50  0000 L CNN
-F 1 "650" H 11220 6855 50  0000 L CNN
+F 1 "1k" H 11220 6855 50  0000 L CNN
 F 2 "Resistor_SMD:R_0603_1608Metric_Pad1.05x0.95mm_HandSolder" V 11080 6900 50  0001 C CNN
 F 3 "~" H 11150 6900 50  0001 C CNN
@@
 	11150 7050 11150 7150
 Wire Wire Line
-	1975 1450 2275 1450
-Wire Wire Line
-	1975 1350 2275 1350
-Wire Wire Line
-	1475 850  1775 850
+	2425 1575 2725 1575
+Wire Wire Line
+	2425 1475 2725 1475
+Wire Wire Line
+	1925 975  2225 975
 $Comp
 L power:+3V3 #PWR0104
@@
 L power:+3V3 #PWR0105
 U 1 1 5E4DF765
-P 1775 850
-F 0 "#PWR0105" H 1775 700 50  0001 C CNN
-F 1 "+3V3" H 1790 1023 50  0000 C CNN
-F 2 "" H 1775 850 50  0001 C CNN
-F 3 "" H 1775 850 50  0001 C CNN
-	1    1775 850
+P 2225 975
+F 0 "#PWR0105" H 2225 825 50  0001 C CNN
+F 1 "+3V3" H 2240 1148 50  0000 C CNN
+F 2 "" H 2225 975 50  0001 C CNN
+F 3 "" H 2225 975 50  0001 C CNN
+	1    2225 975
 	1    0    0    -1
 $EndComp
@@
 L power:GND #PWR0106
 U 1 1 5E4DFD19
-P 2125 1950
-F 0 "#PWR0106" H 2125 1700 50  0001 C CNN
-F 1 "GND" H 2130 1777 50  0000 C CNN
-F 2 "" H 2125 1950 50  0001 C CNN
-F 3 "" H 2125 1950 50  0001 C CNN
-	1    2125 1950
+P 2575 2075
+F 0 "#PWR0106" H 2575 1825 50  0001 C CNN
+F 1 "GND" H 2580 1902 50  0000 C CNN
+F 2 "" H 2575 2075 50  0001 C CNN
+F 3 "" H 2575 2075 50  0001 C CNN
+	1    2575 2075
 	-1   0    0    1
 $EndComp
-Text Label 2275 1350 0    50   ~ 0
+Text Label 2725 1475 0    50   ~ 0
 SWDIO
-Text Label 2275 1450 0    50   ~ 0
+Text Label 2725 1575 0    50   ~ 0
 SWCLK
 Wire Wire Line
-	1475 2050 2125 2050
-Wire Wire Line
-	2125 2050 2125 1950
-Wire Wire Line
-	1975 1150 2275 1150
-Text Label 2275 1150 0    50   ~ 0
+	1925 2175 2575 2175
+Wire Wire Line
+	2575 2175 2575 2075
+Wire Wire Line
+	2425 1275 2725 1275
+Text Label 2725 1275 0    50   ~ 0
 RESET
 $Comp
@@
 Wire Wire Line
 	12000 6450 11650 6450
-Text Notes 11650 7350 0    50   ~ 0
-Rcl = [0.8V * 2500] / Iout(A)
+Text Notes 11600 7400 0    50   ~ 0
+Rcl = [0.8 * 2500] / Iout(A)\nRcl = [0.8 * 2500] / 2A(limit) = 1kohm
 $Comp
 L Switch:SW_Push SW2
@@
 	0    1    1    0
 $EndComp
-Wire Wire Line
-	5450 6000 5300 6000
-Wire Wire Line
-	5450 6100 5300 6100
 Text Label 5200 6400 2    50   ~ 0
 SW_1
@@
 Wire Wire Line
 	5200 5800 5450 5800
-Wire Wire Line
-	5300 5900 5450 5900
 Wire Wire Line
 	5200 5700 5450 5700
@@
 	8900 6850 8600 6850
 Wire Wire Line
-	6650 5900 6850 5900
-Wire Wire Line
 	6650 6000 7100 6000
 Wire Wire Line
@@
 Text Label 7100 6000 0    50   ~ 0
 DIAG_EN
-Text Label 6050 7500 3    50   ~ 0
+Text Label 6050 7850 3    50   ~ 0
 PA_PTT_N
 Text Notes 700  7800 0    50   ~ 0
@@
 Wire Wire Line
 	1700 6600 2150 6600
-Wire Wire Line
-	6150 7500 6150 7850
 Text Label 7100 6200 0    50   ~ 0
 DIAG_4in
-Wire Wire Line
-	6650 5250 6850 5250
 Text Label 7100 6300 0    50   ~ 0
 DIAG_3in
@@
 Wire Wire Line
 	5700 9400 5700 9150
-Text Label 6650 5150 0    50   ~ 0
+Text Label 6850 5150 0    50   ~ 0
 PA_PTT_P
 Text Label 5125 9600 2    50   ~ 0
@@
 P 6850 9150
 F 0 "R21" V 6643 9150 50  0000 C CNN
-F 1 "100" V 6734 9150 50  0000 C CNN
+F 1 "200" V 6734 9150 50  0000 C CNN
 F 2 "Resistor_SMD:R_0603_1608Metric" V 6780 9150 50  0001 C CNN
 F 3 "~" H 6850 9150 50  0001 C CNN
@@
 Wire Wire Line
 	6650 6900 7100 6900
-Wire Wire Line
-	6650 6100 6850 6100
 Wire Wire Line
 	5450 6900 5200 6900
@@
 Text Label 4200 1700 2    50   ~ 0
 HORN
-Text Notes 6425 1900 0    50   ~ 0
-\n\n    Determine quiescent current of rev1 - change rev2 if needed\n    Include diagnostic feedback from load driver to red LED's (user)\n    Include robust software debouncing\nFix Schotky\n\n
-Text Notes 6450 1950 0    50   ~ 0
-Add 2x5 prog header
 $Comp
 L Logan:AdafruitConverter J1
 U 1 1 5EA3B7C5
-P 1475 1450
-F 0 "J1" H 1032 1496 50  0000 R CNN
-F 1 "AdafruitConverter" H 1032 1405 50  0000 R CNN
-F 2 "Connector_PinHeader_1.27mm:PinHeader_2x05_P1.27mm_Vertical_SMD" H 1475 1450 50  0001 C CNN
-F 3 "http://infocenter.arm.com/help/topic/com.arm.doc.ddi0314h/DDI0314H_coresight_components_trm.pdf" V 1125 200 50  0001 C CNN
-	1    1475 1450
+P 1925 1575
+F 0 "J1" H 1482 1621 50  0000 R CNN
+F 1 "AdafruitConverter" H 1482 1530 50  0000 R CNN
+F 2 "Connector_PinHeader_1.27mm:PinHeader_2x05_P1.27mm_Vertical_SMD" H 1925 1575 50  0001 C CNN
+F 3 "http://infocenter.arm.com/help/topic/com.arm.doc.ddi0314h/DDI0314H_coresight_components_trm.pdf" V 1575 325 50  0001 C CNN
+	1    1925 1575
 	1    0    0    -1
 $EndComp
@@
 	6650 5050 6850 5050
 Wire Wire Line
-	6650 4950 6850 4950
-Wire Wire Line
 	6650 6600 7100 6600
 Wire Wire Line
@@
 	-1   0    0    1
 $EndComp
+Text Notes 11100 4625 0    50   ~ 0
+The DIAG_EN pin enables or disables the diagnostic functions.\nIf multiple devices are used,but the ADCresourceis limited in \nthe microcontroller,the MCU can use GPIOs to set DIAG_EN high to\n enable the diagnostics of one device while disabling the \ndiagnostics of the other devices by setting DIAG_EN low. In addition,\nthe device can keep the power consumption to a minimum by \nsetting DIAG_EN and INx low
+Text Notes 6925 8975 0    39   ~ 0
+For current limiting in case of \naccidental shoot through
+Wire Wire Line
+	6650 5150 6850 5150
+Wire Wire Line
+	6050 7500 6050 7850
 $EndSCHEMATC
