File: AddressableV3/AddressableLED.kicad_pcb (KiCad board)
At the start: 2 copper layers, 100 x 22 mm, 77 parts, among them J1 Conn_ARM_JTAG_SWD_10, J2 Conn_01x04_Female, J3 Conn_01x04_Female, Q1 MMBT3904, Q10 MMBT3904, Q11 DMN2041L, Q12 DMN2041L, Q13 DMN2041L, Q14 MMBT3904, Q15 MMBT3904, Q16 MMBT3904, Q17 DMN2041L, Q18 DMN2041L, Q19 DMN2041L, Q2 DMN2041L, Q20 MMBT3904, Q21 MMBT3904, Q22 MMBT3904, Q23 DMN2041L, Q24 DMN2041L, Q25 DMN2041L, Q3 MMBT3904, Q4 DMN2041L, Q5 MMBT3904, Q6 DMN2041L, Q7 MMBT3904, Q8 MMBT3904, Q9 MMBT3904, U1 STM32F030F4Px, U5 MCP1812AT-033_TT

Commit message: Desktop
Parts:
- removed R22, R29: 22, Resistor_SMD:R_0603_1608Metric
- moved D1 51.8 mm to (176.0, 109.2)
- moved D6 51.2 mm to (178.0, 111.5), turned to 180 degrees
- moved D13 48.0 mm to (104.2, 110.0), turned to 180 degrees
- moved D4 46.9 mm to (101.7, 110.0)
- moved D10 46.9 mm to (178.8, 109.2), turned to 180 degrees
- moved D9 43.1 mm to (103.0, 112.0), turned to 180 degrees
- moved D8 35.1 mm to (127.2, 111.8), turned to 180 degrees
- moved D3 28.2 mm to (126.0, 109.5)
- moved D12 26.6 mm to (128.5, 109.5), turned to 180 degrees
- moved D7 1.82 mm to (152.5, 111.5)
- moved D11 1.04 mm to (153.8, 109.0), turned to 180 degrees
- moved D2 0.86 mm to (151.3, 109.0)
Connections:
- J1 pad 10: Net-(J1-Pad10) -> /RESET
- J1 pad 2: Net-(J1-Pad2) -> /SWCLK
- J1 pad 4: Net-(J1-Pad4) -> /SWDIO
- J2 pad 3: /SDA -> Net-(J2-Pad3)
- J2 pad 4: /SCL -> Net-(J2-Pad4)
- J3 pad 3: /SDA -> Net-(J3-Pad3)
- J3 pad 4: /SCL -> Net-(J3-Pad4)
- U1 pad 17: /SCL -> Net-(U1-Pad17)
- U1 pad 18: /SDA -> Net-(U1-Pad18)
Routing:
- net /SDA: track 108.8 -> 0.00 mm
- net /SCL: track 108.1 -> 0.00 mm, vias 2 -> 0
- net Net-(J1-Pad4): track 9.48 -> 0.00 mm
- net /SWDIO: track 7.97 -> 17.4 mm
- net +VDC: track 33.4 -> 29.6 mm
- net /R-_1: track 4.38 -> 1.28 mm
- net /B-_1: track 2.79 -> 0.10 mm
- net Net-(J1-Pad2): track 2.53 -> 0.00 mm
- net /G-_1: track 3.98 -> 1.50 mm
- net /R-_2: track 4.38 -> 6.46 mm
- net /G-_2: track 4.22 -> 2.53 mm
- net /SWCLK: track 9.17 -> 10.6 mm
- net /B-_2: track 2.79 -> 1.79 mm

Commit message: Desktop
Parts:
- removed Q7: MMBT3904, Package_TO_SOT_SMD:SOT-23
- removed R10: 1k, Resistor_SMD:R_0603_1608Metric
- added H1: MountingHole, MountingHole:MountingHole_3.2mm_M3, F.Cu at (115.2, 110.0)
- added H2: MountingHole, MountingHole:MountingHole_3.2mm_M3, F.Cu at (164.8, 110.0)
- added SW1: SW_DIP_x02, Logan:SideMountSwitch, F.Cu at (133.9, 119.5)
- added SW2: SW_DIP_x02, Logan:SideMountSwitch, F.Cu at (139.4, 119.5)
- added SW3: SW_DIP_x02, Logan:SideMountSwitch, F.Cu at (144.9, 119.5)
- C1: moved to B.Cu
- J2: value Conn_01x04_Female -> Conn_01x02_Female; footprint AddressableLED:1.5mmHole -> Connector_JST:JST_VH_B2P-VH_1x02_P3.96mm_Vertical
- J3: value Conn_01x04_Female -> Conn_01x02_Female; footprint AddressableLED:1.5mmHoleMirror -> Connector_JST:JST_VH_B2P-VH_1x02_P3.96mm_Vertical
- R21: value 22 -> 0
- moved J3 65.7 mm to (118.0, 88.2), turned to 0 degrees
- moved J2 65.0 mm to (164.9, 105.7), turned to 90 degrees
- moved C1 16.2 mm to (149.2, 107.3), turned to 90 degrees
- moved C2 2.48 mm to (145.5, 110.0)
- moved U5 2.45 mm to (148.2, 110.2)
- moved D13 1.32 mm to (103.7, 108.8)
- moved D4 1.27 mm to (101.3, 108.8)
- moved D9 1.03 mm to (102.5, 111.1)
- moved D8 0.25 mm to (127.5, 111.8)
- moved R21 0.21 mm to (138.8, 104.2)
Connections:
- C2 pad 1: Net-(C2-Pad1) -> +3V3
- J1 pad 10: /RESET -> Net-(J1-Pad10)
- J1 pad 2: /SWCLK -> /SWDIO
- J1 pad 4: /SWDIO -> /SWCLK
- U5 pad 1: Net-(Q7-Pad3) -> +3V3
Routing:
- net +VDC: track 29.6 -> 14.3 mm, vias 11 -> 12
- net +3V3: track 31.0 -> 23.5 mm
- net Net-(Q7-Pad3): track 7.35 -> 0.00 mm
- net Net-(Q11-Pad2): track 6.58 -> 0.00 mm
- net /SWDIO: track 17.4 -> 12.0 mm
- net /SWCLK: track 10.6 -> 15.4 mm
- net /G-_4: track 4.22 -> 0.14 mm
- net Net-(C2-Pad1): track 3.13 -> 0.00 mm
- net Net-(Q11-Pad1): track 8.40 -> 5.46 mm
- net Net-(Q20-Pad3): track 14.6 -> 12.3 mm
- net /B-_2: track 1.79 -> 0.00 mm
- net GND: track 12.2 -> 13.4 mm, vias 91 -> 81
- net Net-(J1-Pad10): track 5.42 -> 4.31 mm
- net /R-_3: vias 0 -> 1
- added copper zone on B.Cu, net +3V3
- added copper zone on F.Cu, net +3V3

Commit message: Desktop
Parts:
- removed U5: MCP1812AT-033_TT, Package_TO_SOT_SMD:SOT-23
- added C3: 22u, Capacitor_SMD:C_0603_1608Metric, B.Cu at (145.6, 110.0)
- added C6: 22u, Capacitor_SMD:C_0603_1608Metric, F.Cu at (109.7, 104.3)
- added C7: 22u, Capacitor_SMD:C_0603_1608Metric, F.Cu at (111.2, 104.3)
- added C8: 22u, Capacitor_SMD:C_0603_1608Metric, F.Cu at (117.5, 110.2)
- added C9: 22u, Capacitor_SMD:C_0603_1608Metric, F.Cu at (114.2, 110.0)
- added L1: 2.2u, Inductor_SMD:L_Coilcraft_XxL4020, F.Cu at (111.0, 108.3)
- added R10: 10k, Resistor_SMD:R_0603_1608Metric, F.Cu at (117.7, 106.9)
- added R22: 1k, Resistor_SMD:R_0603_1608Metric, B.Cu at (146.6, 116.7)
- added R29: 0, Resistor_SMD:R_0603_1608Metric, B.Cu at (138.9, 104.3)
- added U2: MCP1812AT-033_TT, Package_TO_SOT_SMD:SOT-23, B.Cu at (148.4, 110.3)
- added U3: STM32F030F4Px, Package_SO:TSSOP-20_4.4x6.5mm_P0.65mm, B.Cu at (140.0, 109.8)
- C1: value 22u -> 0.1u; moved to F.Cu
- D5: moved to B.Cu
- J2: footprint Connector_JST:JST_VH_B2P-VH_1x02_P3.96mm_Vertical -> AddressableLED:1.5mmHole
- J3: footprint Connector_JST:JST_VH_B2P-VH_1x02_P3.96mm_Vertical -> AddressableLED:1.5mmHoleMirror
- R21: value 0 -> 36k; moved to F.Cu
- R30: value 220 -> 10k; moved to B.Cu
- R9: moved to F.Cu
- U1: value STM32F030F4Px -> TPS563200; footprint Package_SO:TSSOP-20_4.4x6.5mm_P0.65mm -> Package_TO_SOT_SMD:SOT-23-6; moved to F.Cu
- moved J3 65.7 mm to (180.0, 110.0), turned to 180 degrees
- moved J2 65.0 mm to (100.0, 110.0), turned to 0 degrees
- moved C1 34.4 mm to (114.8, 106.6), turned to 180 degrees
- moved R9 31.2 mm to (113.8, 101.3)
- moved H1 28.9 mm to (91.5, 93.5)
- moved U1 25.9 mm to (114.8, 104.0), turned to 0 degrees
- moved R21 23.3 mm to (116.0, 109.0), turned to 270 degrees
- moved R30 12.2 mm to (145.1, 101.4), turned to 0 degrees
- moved C2 5.72 mm to (149.9, 113.7)
- moved D5 3.17 mm to (143.2, 116.7), turned to 180 degrees
- moved SW3 0.80 mm to (145.7, 119.5)
- moved D3 0.77 mm to (126.3, 108.8)
- moved D12 0.73 mm to (128.7, 108.8)
- moved Q10 0.70 mm to (106.7, 106.8)
- moved Q13 0.70 mm to (106.7, 110.4)
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Connections:
- net /RESET renamed Net-(R10-Pad2)
- C1 pad 1: +VDC -> Net-(C1-Pad1)
- C1 pad 2: GND -> Net-(C1-Pad2)
- C2 pad 1: +3V3 -> 3V8
- D1 pad 2: +VDC -> 3V8
- D10 pad 2: +VDC -> 3V8
- D11 pad 2: +VDC -> 3V8
- D12 pad 2: +VDC -> 3V8
- D13 pad 2: +VDC -> 3V8
- D2 pad 2: +VDC -> 3V8
- D3 pad 2: +VDC -> 3V8
- D4 pad 2: +VDC -> 3V8
- D6 pad 2: +VDC -> 3V8
- D7 pad 2: +VDC -> 3V8
- D8 pad 2: +VDC -> 3V8
- D9 pad 2: +VDC -> 3V8
- J1 pad 2: /SWDIO -> /Microcontroller/SWDIO
- J1 pad 4: /SWCLK -> /Microcontroller/SWCLK
- J2 pad 1: +VDC -> VDC
- J3 pad 1: +VDC -> VDC
- R21 pad 2: Net-(J1-Pad10) -> 3V8
- R30 pad 1: Net-(D5-Pad1) -> Net-(R30-Pad1)
- R9 pad 1: Net-(R9-Pad1) -> VDC
- R9 pad 2: GND -> Net-(R9-Pad2)
- SW3 pad 2: Net-(SW3-Pad2) -> Net-(SW3-Pad1)
- SW3 pad 4: Net-(SW3-Pad4) -> Net-(SW3-Pad3)
- U1 pad 1: Net-(R9-Pad1) -> GND
- U1 pad 2: Net-(U1-Pad2) -> Net-(C1-Pad2)
- U1 pad 3: Net-(U1-Pad3) -> VDC
- U1 pad 5: +3V3 -> Net-(R9-Pad2)
- U1 pad 6: Net-(U1-Pad6) -> Net-(C1-Pad1)
Routing:
- net VDC: track 0.00 -> 35.6 mm
- net /SWCLK: track 15.4 -> 0.00 mm, vias 1 -> 0
- net /Microcontroller/SWCLK: track 0.00 -> 15.4 mm, vias 0 -> 1
- net +VDC: track 14.3 -> 0.00 mm, vias 12 -> 0
- net /SWDIO: track 12.0 -> 0.00 mm, vias 1 -> 0
- net /Microcontroller/SWDIO: track 0.00 -> 12.0 mm, vias 0 -> 1
- net 3V8: track 0.00 -> 10.8 mm, vias 0 -> 12
- net Net-(R9-Pad1): track 10.4 -> 0.00 mm
- net Net-(R30-Pad1): track 0.00 -> 10.4 mm
- net Net-(Q15-Pad3): track 7.58 -> 0.00 mm
- net Net-(C1-Pad2): track 0.00 -> 6.86 mm
- net GND: track 13.4 -> 19.8 mm, vias 81 -> 82
- net Net-(Q15-Pad1): track 6.36 -> 0.00 mm
- net /R-_2: track 6.46 -> 1.28 mm
- net Net-(C1-Pad1): track 0.00 -> 4.61 mm
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- added copper zone on B.Cu, net 3V8
- removed copper zone on B.Cu, net +VDC
Other:
- board text removed: "SCL"
- board text removed: "SDA"

Commit message: Desktop
Parts:
- removed R9: 10k, Resistor_SMD:R_0603_1608Metric
- C1, C6, C7, C8, C9, L1, R10, R21, U1: moved to B.Cu
- moved R21 22.7 mm to (100.9, 126.0), turned to 180 degrees
- moved C7 18.4 mm to (99.2, 118.2), turned to 270 degrees
- moved C6 16.4 mm to (101.0, 118.2)
- moved U1 16.1 mm to (102.5, 114.4), turned to 90 degrees
- moved R10 15.0 mm to (103.3, 111.3), turned to 180 degrees
- moved C1 9.61 mm to (106.5, 111.3), turned to 0 degrees
- moved L1 8.18 mm to (107.9, 115.9), turned to 0 degrees
- moved C8 7.92 mm to (113.2, 116.7)
- moved C9 7.34 mm to (111.2, 116.8)
Connections:
- U1 pad 5: Net-(R9-Pad2) -> VDC
Routing:
- net VDC: track 35.6 -> 2.14 mm
- net GND: track 19.8 -> 12.2 mm, vias 82 -> 83
- net 3V8: track 10.8 -> 15.5 mm
- net Net-(C1-Pad2): track 6.86 -> 10.4 mm
- net Net-(R10-Pad2): track 5.11 -> 2.70 mm
- net Net-(C1-Pad1): track 4.61 -> 3.46 mm
- added copper zone on B.Cu, net VDC

Commit message: Desktop
Parts:
- removed C1: 0.1u, Capacitor_SMD:C_0603_1608Metric
- removed C6, C7, C8, C9: 22u, Capacitor_SMD:C_0603_1608Metric
- removed J3: Conn_01x02_Female, AddressableLED:1.5mmHoleMirror
- removed L1: 2.2u, Inductor_SMD:L_Coilcraft_XxL4020
- added R9: 10k, Resistor_SMD:R_0603_1608Metric, F.Cu at (138.0, 117.3)
- added REF**: VIA-0.6mm, Logan:VIA-0.6mm, F.Cu at (170.6, 119.7)
- added REF**: VIA-0.6mm, Logan:VIA-0.6mm, F.Cu at (161.6, 119.7)
- added REF**: VIA-0.6mm, Logan:VIA-0.6mm, F.Cu at (120.2, 115.8)
- added REF**: VIA-0.6mm, Logan:VIA-0.6mm, F.Cu at (119.2, 115.8)
- added REF**: VIA-0.6mm, Logan:VIA-0.6mm, F.Cu at (118.2, 115.8)
- added REF**: VIA-0.6mm, Logan:VIA-0.6mm, F.Cu at (117.2, 115.8)
- added REF**: VIA-0.6mm, Logan:VIA-0.6mm, F.Cu at (116.2, 115.8)
- added REF**: VIA-0.6mm, Logan:VIA-0.6mm, F.Cu at (115.2, 115.8)
- added REF**: VIA-0.6mm, Logan:VIA-0.6mm, F.Cu at (114.2, 115.8)
- added REF**: VIA-0.6mm, Logan:VIA-0.6mm, F.Cu at (113.2, 115.8)
- added REF**: VIA-0.6mm, Logan:VIA-0.6mm, F.Cu at (112.2, 115.8)
- added REF**: VIA-0.6mm, Logan:VIA-0.6mm, F.Cu at (111.2, 115.8)
- added REF**: VIA-0.6mm, Logan:VIA-0.6mm, F.Cu at (160.6, 119.7)
- added REF**: VIA-0.6mm, Logan:VIA-0.6mm, F.Cu at (110.2, 115.8)
- added REF**: VIA-0.6mm, Logan:VIA-0.6mm, F.Cu at (168.6, 114.7)
- added REF**: VIA-0.6mm, Logan:VIA-0.6mm, F.Cu at (167.6, 114.7)
- added REF**: VIA-0.6mm, Logan:VIA-0.6mm, F.Cu at (166.6, 114.7)
- added REF**: VIA-0.6mm, Logan:VIA-0.6mm, F.Cu at (165.6, 114.7)
- added REF**: VIA-0.6mm, Logan:VIA-0.6mm, F.Cu at (164.6, 114.7)
- added REF**: VIA-0.6mm, Logan:VIA-0.6mm, F.Cu at (163.6, 114.7)
- added REF**: VIA-0.6mm, Logan:VIA-0.6mm, F.Cu at (162.6, 114.7)
- added REF**: VIA-0.6mm, Logan:VIA-0.6mm, F.Cu at (161.6, 114.7)
- added REF**: VIA-0.6mm, Logan:VIA-0.6mm, F.Cu at (160.6, 114.7)
- added REF**: VIA-0.6mm, Logan:VIA-0.6mm, F.Cu at (170.6, 118.7)
- added REF**: VIA-0.6mm, Logan:VIA-0.6mm, F.Cu at (120.2, 114.8)
- added REF**: VIA-0.6mm, Logan:VIA-0.6mm, F.Cu at (168.6, 113.7)
- added REF**: VIA-0.6mm, Logan:VIA-0.6mm, F.Cu at (167.6, 113.7)
- added REF**: VIA-0.6mm, Logan:VIA-0.6mm, F.Cu at (166.6, 113.7)
- added REF**: VIA-0.6mm, Logan:VIA-0.6mm, F.Cu at (165.6, 113.7)
- added REF**: VIA-0.6mm, Logan:VIA-0.6mm, F.Cu at (164.6, 113.7)
- added REF**: VIA-0.6mm, Logan:VIA-0.6mm, F.Cu at (163.6, 113.7)
- added REF**: VIA-0.6mm, Logan:VIA-0.6mm, F.Cu at (162.6, 113.7)
- added REF**: VIA-0.6mm, Logan:VIA-0.6mm, F.Cu at (161.6, 113.7)
- added REF**: VIA-0.6mm, Logan:VIA-0.6mm, F.Cu at (160.6, 113.7)
- added REF**: VIA-0.6mm, Logan:VIA-0.6mm, F.Cu at (169.6, 118.7)
- added REF**: VIA-0.6mm, Logan:VIA-0.6mm, F.Cu at (120.2, 113.8)
- added REF**: VIA-0.6mm, Logan:VIA-0.6mm, F.Cu at (168.6, 112.7)
- added REF**: VIA-0.6mm, Logan:VIA-0.6mm, F.Cu at (167.6, 112.7)
- added REF**: VIA-0.6mm, Logan:VIA-0.6mm, F.Cu at (166.6, 112.7)
- added REF**: VIA-0.6mm, Logan:VIA-0.6mm, F.Cu at (165.6, 112.7)
- added REF**: VIA-0.6mm, Logan:VIA-0.6mm, F.Cu at (164.6, 112.7)
- added REF**: VIA-0.6mm, Logan:VIA-0.6mm, F.Cu at (163.6, 112.7)
- added REF**: VIA-0.6mm, Logan:VIA-0.6mm, F.Cu at (162.6, 112.7)
- added REF**: VIA-0.6mm, Logan:VIA-0.6mm, F.Cu at (161.6, 112.7)
- added REF**: VIA-0.6mm, Logan:VIA-0.6mm, F.Cu at (160.6, 112.7)
- added REF**: VIA-0.6mm, Logan:VIA-0.6mm, F.Cu at (168.6, 118.7)
- added REF**: VIA-0.6mm, Logan:VIA-0.6mm, F.Cu at (120.2, 112.8)
- added REF**: VIA-0.6mm, Logan:VIA-0.6mm, F.Cu at (168.6, 111.7)
- added REF**: VIA-0.6mm, Logan:VIA-0.6mm, F.Cu at (167.6, 111.7)
- added REF**: VIA-0.6mm, Logan:VIA-0.6mm, F.Cu at (166.6, 111.7)
- added REF**: VIA-0.6mm, Logan:VIA-0.6mm, F.Cu at (162.6, 111.7)
- added REF**: VIA-0.6mm, Logan:VIA-0.6mm, F.Cu at (161.6, 111.7)
- added REF**: VIA-0.6mm, Logan:VIA-0.6mm, F.Cu at (160.6, 111.7)
- added REF**: VIA-0.6mm, Logan:VIA-0.6mm, F.Cu at (120.2, 111.8)
- added REF**: VIA-0.6mm, Logan:VIA-0.6mm, F.Cu at (168.6, 110.7)
- added REF**: VIA-0.6mm, Logan:VIA-0.6mm, F.Cu at (167.6, 110.7)
- added REF**: VIA-0.6mm, Logan:VIA-0.6mm, F.Cu at (167.6, 118.7)
- added REF**: VIA-0.6mm, Logan:VIA-0.6mm, F.Cu at (161.6, 110.7)
- added REF**: VIA-0.6mm, Logan:VIA-0.6mm, F.Cu at (160.6, 110.7)
- added REF**: VIA-0.6mm, Logan:VIA-0.6mm, F.Cu at (120.2, 110.8)
- added REF**: VIA-0.6mm, Logan:VIA-0.6mm, F.Cu at (170.6, 114.7)
- added REF**: VIA-0.6mm, Logan:VIA-0.6mm, F.Cu at (169.6, 114.7)
- added REF**: VIA-0.6mm, Logan:VIA-0.6mm, F.Cu at (119.2, 114.8)
- added REF**: VIA-0.6mm, Logan:VIA-0.6mm, F.Cu at (118.2, 114.8)
- added REF**: VIA-0.6mm, Logan:VIA-0.6mm, F.Cu at (117.2, 114.8)
- added REF**: VIA-0.6mm, Logan:VIA-0.6mm, F.Cu at (116.2, 114.8)
- added REF**: VIA-0.6mm, Logan:VIA-0.6mm, F.Cu at (115.2, 114.8)
- added REF**: VIA-0.6mm, Logan:VIA-0.6mm, F.Cu at (166.6, 118.7)
- added REF**: VIA-0.6mm, Logan:VIA-0.6mm, F.Cu at (170.6, 113.7)
- added REF**: VIA-0.6mm, Logan:VIA-0.6mm, F.Cu at (169.6, 113.7)
- added REF**: VIA-0.6mm, Logan:VIA-0.6mm, F.Cu at (119.2, 113.8)
- added REF**: VIA-0.6mm, Logan:VIA-0.6mm, F.Cu at (118.2, 113.8)
- added REF**: VIA-0.6mm, Logan:VIA-0.6mm, F.Cu at (117.2, 113.8)
- added REF**: VIA-0.6mm, Logan:VIA-0.6mm, F.Cu at (116.2, 113.8)
- added REF**: VIA-0.6mm, Logan:VIA-0.6mm, F.Cu at (115.2, 113.8)
- added REF**: VIA-0.6mm, Logan:VIA-0.6mm, F.Cu at (170.6, 112.7)
- added REF**: VIA-0.6mm, Logan:VIA-0.6mm, F.Cu at (169.6, 112.7)
- added REF**: VIA-0.6mm, Logan:VIA-0.6mm, F.Cu at (119.2, 112.8)
- added REF**: VIA-0.6mm, Logan:VIA-0.6mm, F.Cu at (165.6, 118.7)
- added REF**: VIA-0.6mm, Logan:VIA-0.6mm, F.Cu at (118.2, 112.8)
- added REF**: VIA-0.6mm, Logan:VIA-0.6mm, F.Cu at (117.2, 112.8)
- added REF**: VIA-0.6mm, Logan:VIA-0.6mm, F.Cu at (116.2, 112.8)
- added REF**: VIA-0.6mm, Logan:VIA-0.6mm, F.Cu at (115.2, 112.8)
- added REF**: VIA-0.6mm, Logan:VIA-0.6mm, F.Cu at (170.6, 111.7)
- added REF**: VIA-0.6mm, Logan:VIA-0.6mm, F.Cu at (169.6, 111.7)
- added REF**: VIA-0.6mm, Logan:VIA-0.6mm, F.Cu at (119.2, 111.8)
- added REF**: VIA-0.6mm, Logan:VIA-0.6mm, F.Cu at (118.2, 111.8)
- added REF**: VIA-0.6mm, Logan:VIA-0.6mm, F.Cu at (117.2, 111.8)
- added REF**: VIA-0.6mm, Logan:VIA-0.6mm, F.Cu at (170.6, 110.7)
- added REF**: VIA-0.6mm, Logan:VIA-0.6mm, F.Cu at (164.6, 118.7)
- added REF**: VIA-0.6mm, Logan:VIA-0.6mm, F.Cu at (169.6, 110.7)
- added REF**: VIA-0.6mm, Logan:VIA-0.6mm, F.Cu at (119.2, 110.8)
- added REF**: VIA-0.6mm, Logan:VIA-0.6mm, F.Cu at (118.2, 110.8)
- added REF**: VIA-0.6mm, Logan:VIA-0.6mm, F.Cu at (117.2, 110.8)
- added REF**: VIA-0.6mm, Logan:VIA-0.6mm, F.Cu at (114.2, 114.8)
- added REF**: VIA-0.6mm, Logan:VIA-0.6mm, F.Cu at (113.2, 114.8)
- added REF**: VIA-0.6mm, Logan:VIA-0.6mm, F.Cu at (112.2, 114.8)
- added REF**: VIA-0.6mm, Logan:VIA-0.6mm, F.Cu at (111.2, 114.8)
- added REF**: VIA-0.6mm, Logan:VIA-0.6mm, F.Cu at (110.2, 114.8)
- added REF**: VIA-0.6mm, Logan:VIA-0.6mm, F.Cu at (114.2, 113.8)
- added REF**: VIA-0.6mm, Logan:VIA-0.6mm, F.Cu at (163.6, 118.7)
- added REF**: VIA-0.6mm, Logan:VIA-0.6mm, F.Cu at (113.2, 113.8)
- added REF**: VIA-0.6mm, Logan:VIA-0.6mm, F.Cu at (112.2, 113.8)
- added REF**: VIA-0.6mm, Logan:VIA-0.6mm, F.Cu at (111.2, 113.8)
- added REF**: VIA-0.6mm, Logan:VIA-0.6mm, F.Cu at (110.2, 113.8)
- added REF**: VIA-0.6mm, Logan:VIA-0.6mm, F.Cu at (114.2, 112.8)
- added REF**: VIA-0.6mm, Logan:VIA-0.6mm, F.Cu at (113.2, 112.8)
- added REF**: VIA-0.6mm, Logan:VIA-0.6mm, F.Cu at (112.2, 112.8)
- added REF**: VIA-0.6mm, Logan:VIA-0.6mm, F.Cu at (111.2, 112.8)
- added REF**: VIA-0.6mm, Logan:VIA-0.6mm, F.Cu at (110.2, 112.8)
- added REF**: VIA-0.6mm, Logan:VIA-0.6mm, F.Cu at (112.2, 111.8)
- added REF**: VIA-0.6mm, Logan:VIA-0.6mm, F.Cu at (169.6, 119.7)
- added REF**: VIA-0.6mm, Logan:VIA-0.6mm, F.Cu at (162.6, 118.7)
- added REF**: VIA-0.6mm, Logan:VIA-0.6mm, F.Cu at (111.2, 111.8)
- added REF**: VIA-0.6mm, Logan:VIA-0.6mm, F.Cu at (110.2, 111.8)
- added REF**: VIA-0.6mm, Logan:VIA-0.6mm, F.Cu at (112.2, 110.8)
- added REF**: VIA-0.6mm, Logan:VIA-0.6mm, F.Cu at (111.2, 110.8)
- added REF**: VIA-0.6mm, Logan:VIA-0.6mm, F.Cu at (110.2, 110.8)
- added REF**: VIA-0.6mm, Logan:VIA-0.6mm, F.Cu at (161.6, 118.7)
- added REF**: VIA-0.6mm, Logan:VIA-0.6mm, F.Cu at (160.6, 118.7)
- added REF**: VIA-0.6mm, Logan:VIA-0.6mm, F.Cu at (170.6, 117.7)
- added REF**: VIA-0.6mm, Logan:VIA-0.6mm, F.Cu at (169.6, 117.7)
- added REF**: VIA-0.6mm, Logan:VIA-0.6mm, F.Cu at (168.6, 117.7)
- added REF**: VIA-0.6mm, Logan:VIA-0.6mm, F.Cu at (167.6, 117.7)
- added REF**: VIA-0.6mm, Logan:VIA-0.6mm, F.Cu at (166.6, 117.7)
- added REF**: VIA-0.6mm, Logan:VIA-0.6mm, F.Cu at (165.6, 117.7)
- added REF**: VIA-0.6mm, Logan:VIA-0.6mm, F.Cu at (164.6, 117.7)
- added REF**: VIA-0.6mm, Logan:VIA-0.6mm, F.Cu at (168.6, 119.7)
- added REF**: VIA-0.6mm, Logan:VIA-0.6mm, F.Cu at (163.6, 117.7)
- added REF**: VIA-0.6mm, Logan:VIA-0.6mm, F.Cu at (162.6, 117.7)
- added REF**: VIA-0.6mm, Logan:VIA-0.6mm, F.Cu at (161.6, 117.7)
- added REF**: VIA-0.6mm, Logan:VIA-0.6mm, F.Cu at (160.6, 117.7)
- added REF**: VIA-0.6mm, Logan:VIA-0.6mm, F.Cu at (170.6, 116.7)
- added REF**: VIA-0.6mm, Logan:VIA-0.6mm, F.Cu at (169.6, 116.7)
- added REF**: VIA-0.6mm, Logan:VIA-0.6mm, F.Cu at (168.6, 116.7)
- added REF**: VIA-0.6mm, Logan:VIA-0.6mm, F.Cu at (167.6, 116.7)
- added REF**: VIA-0.6mm, Logan:VIA-0.6mm, F.Cu at (166.6, 116.7)
- added REF**: VIA-0.6mm, Logan:VIA-0.6mm, F.Cu at (165.6, 116.7)
- added REF**: VIA-0.6mm, Logan:VIA-0.6mm, F.Cu at (167.6, 119.7)
- added REF**: VIA-0.6mm, Logan:VIA-0.6mm, F.Cu at (164.6, 116.7)
- added REF**: VIA-0.6mm, Logan:VIA-0.6mm, F.Cu at (163.6, 116.7)
- added REF**: VIA-0.6mm, Logan:VIA-0.6mm, F.Cu at (162.6, 116.7)
- added REF**: VIA-0.6mm, Logan:VIA-0.6mm, F.Cu at (161.6, 116.7)
- added REF**: VIA-0.6mm, Logan:VIA-0.6mm, F.Cu at (160.6, 116.7)
- added REF**: VIA-0.6mm, Logan:VIA-0.6mm, F.Cu at (170.6, 115.7)
- added REF**: VIA-0.6mm, Logan:VIA-0.6mm, F.Cu at (169.6, 115.7)
- added REF**: VIA-0.6mm, Logan:VIA-0.6mm, F.Cu at (168.6, 115.7)
- added REF**: VIA-0.6mm, Logan:VIA-0.6mm, F.Cu at (167.6, 115.7)
- added REF**: VIA-0.6mm, Logan:VIA-0.6mm, F.Cu at (166.6, 115.7)
- added REF**: VIA-0.6mm, Logan:VIA-0.6mm, F.Cu at (166.6, 119.7)
- added REF**: VIA-0.6mm, Logan:VIA-0.6mm, F.Cu at (165.6, 115.7)
- added REF**: VIA-0.6mm, Logan:VIA-0.6mm, F.Cu at (164.6, 115.7)
- added REF**: VIA-0.6mm, Logan:VIA-0.6mm, F.Cu at (163.6, 115.7)
- added REF**: VIA-0.6mm, Logan:VIA-0.6mm, F.Cu at (162.6, 115.7)
- added REF**: VIA-0.6mm, Logan:VIA-0.6mm, F.Cu at (161.6, 115.7)
- added REF**: VIA-0.6mm, Logan:VIA-0.6mm, F.Cu at (160.6, 115.7)
- added REF**: VIA-0.6mm, Logan:VIA-0.6mm, F.Cu at (120.2, 119.8)
- added REF**: VIA-0.6mm, Logan:VIA-0.6mm, F.Cu at (119.2, 119.8)
- added REF**: VIA-0.6mm, Logan:VIA-0.6mm, F.Cu at (118.2, 119.8)
- added REF**: VIA-0.6mm, Logan:VIA-0.6mm, F.Cu at (117.2, 119.8)
- added REF**: VIA-0.6mm, Logan:VIA-0.6mm, F.Cu at (165.6, 119.7)
- added REF**: VIA-0.6mm, Logan:VIA-0.6mm, F.Cu at (116.2, 119.8)
- added REF**: VIA-0.6mm, Logan:VIA-0.6mm, F.Cu at (115.2, 119.8)
- added REF**: VIA-0.6mm, Logan:VIA-0.6mm, F.Cu at (114.2, 119.8)
- added REF**: VIA-0.6mm, Logan:VIA-0.6mm, F.Cu at (113.2, 119.8)
- added REF**: VIA-0.6mm, Logan:VIA-0.6mm, F.Cu at (112.2, 119.8)
- added REF**: VIA-0.6mm, Logan:VIA-0.6mm, F.Cu at (111.2, 119.8)
- added REF**: VIA-0.6mm, Logan:VIA-0.6mm, F.Cu at (110.2, 119.8)
- added REF**: VIA-0.6mm, Logan:VIA-0.6mm, F.Cu at (120.2, 118.8)
- added REF**: VIA-0.6mm, Logan:VIA-0.6mm, F.Cu at (119.2, 118.8)
- added REF**: VIA-0.6mm, Logan:VIA-0.6mm, F.Cu at (118.2, 118.8)
- added REF**: VIA-0.6mm, Logan:VIA-0.6mm, F.Cu at (164.6, 119.7)
- added REF**: VIA-0.6mm, Logan:VIA-0.6mm, F.Cu at (117.2, 118.8)
- added REF**: VIA-0.6mm, Logan:VIA-0.6mm, F.Cu at (116.2, 118.8)
- added REF**: VIA-0.6mm, Logan:VIA-0.6mm, F.Cu at (115.2, 118.8)
- added REF**: VIA-0.6mm, Logan:VIA-0.6mm, F.Cu at (114.2, 118.8)
- added REF**: VIA-0.6mm, Logan:VIA-0.6mm, F.Cu at (113.2, 118.8)
- added REF**: VIA-0.6mm, Logan:VIA-0.6mm, F.Cu at (112.2, 118.8)
- added REF**: VIA-0.6mm, Logan:VIA-0.6mm, F.Cu at (111.2, 118.8)
- added REF**: VIA-0.6mm, Logan:VIA-0.6mm, F.Cu at (110.2, 118.8)
- added REF**: VIA-0.6mm, Logan:VIA-0.6mm, F.Cu at (120.2, 117.8)
- added REF**: VIA-0.6mm, Logan:VIA-0.6mm, F.Cu at (119.2, 117.8)
- added REF**: VIA-0.6mm, Logan:VIA-0.6mm, F.Cu at (163.6, 119.7)
- added REF**: VIA-0.6mm, Logan:VIA-0.6mm, F.Cu at (118.2, 117.8)
- added REF**: VIA-0.6mm, Logan:VIA-0.6mm, F.Cu at (117.2, 117.8)
- added REF**: VIA-0.6mm, Logan:VIA-0.6mm, F.Cu at (116.2, 117.8)
- added REF**: VIA-0.6mm, Logan:VIA-0.6mm, F.Cu at (115.2, 117.8)
- added REF**: VIA-0.6mm, Logan:VIA-0.6mm, F.Cu at (114.2, 117.8)
- added REF**: VIA-0.6mm, Logan:VIA-0.6mm, F.Cu at (113.2, 117.8)
- added REF**: VIA-0.6mm, Logan:VIA-0.6mm, F.Cu at (112.2, 117.8)
- added REF**: VIA-0.6mm, Logan:VIA-0.6mm, F.Cu at (111.2, 117.8)
- added REF**: VIA-0.6mm, Logan:VIA-0.6mm, F.Cu at (110.2, 117.8)
- added REF**: VIA-0.6mm, Logan:VIA-0.6mm, F.Cu at (120.2, 116.8)
- added REF**: VIA-0.6mm, Logan:VIA-0.6mm, F.Cu at (162.6, 119.7)
- added REF**: VIA-0.6mm, Logan:VIA-0.6mm, F.Cu at (119.2, 116.8)
- added REF**: VIA-0.6mm, Logan:VIA-0.6mm, F.Cu at (118.2, 116.8)
- added REF**: VIA-0.6mm, Logan:VIA-0.6mm, F.Cu at (117.2, 116.8)
- added REF**: VIA-0.6mm, Logan:VIA-0.6mm, F.Cu at (116.2, 116.8)
- added REF**: VIA-0.6mm, Logan:VIA-0.6mm, F.Cu at (115.2, 116.8)
- added REF**: VIA-0.6mm, Logan:VIA-0.6mm, F.Cu at (114.2, 116.8)
- added REF**: VIA-0.6mm, Logan:VIA-0.6mm, F.Cu at (113.2, 116.8)
- added REF**: VIA-0.6mm, Logan:VIA-0.6mm, F.Cu at (112.2, 116.8)
- added REF**: VIA-0.6mm, Logan:VIA-0.6mm, F.Cu at (111.2, 116.8)
- added REF**: VIA-0.6mm, Logan:VIA-0.6mm, F.Cu at (110.2, 116.8)
- R21: value 36k -> 10k; moved to F.Cu
- U1: value TPS563200 -> LoganSWModule; footprint Package_TO_SOT_SMD:SOT-23-6 -> Logan:Logan_SWmodule
- moved J2 92.1 mm to (192.1, 110.0)
- moved U1 67.5 mm to (169.8, 110.0), turned to 0 degrees
- moved R21 43.3 mm to (143.3, 117.3), turned to 0 degrees
- moved R10 32.0 mm to (134.8, 117.3)
- moved H1 28.5 mm to (114.7, 110.0)
- moved D5 0.70 mm to (143.2, 116.0)
- moved R22 0.70 mm to (146.5, 116.0)
- moved J1 0.70 mm to (140.1, 104.3)
- moved D6 0.64 mm to (177.5, 111.1)
- moved D1 0.54 mm to (176.3, 108.8)
- moved D10 0.45 mm to (178.7, 108.8)
- moved D7 0.40 mm to (152.5, 111.1), turned to 180 degrees
- moved D11 0.21 mm to (153.7, 108.8)
- moved D2 0.20 mm to (151.3, 108.8)
Connections:
- R1 pad 1: /B -> B
- R10 pad 1: GND -> +3V3
- R10 pad 2: Net-(R10-Pad2) -> /Microcontroller/SW2
- R11 pad 1: /G -> G
- R12 pad 1: /G -> G
- R14 pad 1: /G -> G
- R15 pad 1: /G -> G
- R17 pad 1: /R -> R
- R2 pad 1: /B -> B
- R21 pad 1: Net-(R10-Pad2) -> +3V3
- R21 pad 2: 3V8 -> /Microcontroller/SW3
- R23 pad 1: /R -> R
- R24 pad 1: /R -> R
- R25 pad 1: /R -> R
- R3 pad 1: /B -> B
- R7 pad 1: /B -> B
- SW1 pad 1: Net-(SW1-Pad1) -> GND
- SW1 pad 2: Net-(SW1-Pad2) -> GND
- SW1 pad 3: Net-(SW1-Pad3) -> /Microcontroller/SW1
- SW1 pad 4: Net-(SW1-Pad4) -> /Microcontroller/SW1
- SW2 pad 1: Net-(SW2-Pad1) -> GND
- SW2 pad 2: Net-(SW2-Pad2) -> GND
- SW2 pad 3: Net-(SW2-Pad3) -> /Microcontroller/SW2
- SW2 pad 4: Net-(SW2-Pad4) -> /Microcontroller/SW2
- SW3 pad 1: Net-(SW3-Pad1) -> GND
- SW3 pad 2: Net-(SW3-Pad1) -> GND
- SW3 pad 3: Net-(SW3-Pad3) -> /Microcontroller/SW3
- SW3 pad 4: Net-(SW3-Pad3) -> /Microcontroller/SW3
- U1 pad 2: Net-(C1-Pad2) -> GND
- U1 pad 4: Net-(R10-Pad2) -> VDC
- U1 pad 5: VDC -> 3V8
- U1 pad 6: Net-(C1-Pad1) -> 3V8
- U3 pad 17: Net-(U3-Pad17) -> /Microcontroller/SW3
- U3 pad 18: Net-(U3-Pad18) -> /Microcontroller/SW1
- U3 pad 2: Net-(U3-Pad2) -> /Microcontroller/SW2
Routing:
- net R: track 0.00 -> 100.4 mm, vias 0 -> 4
- net /R: track 100.3 -> 0.00 mm, vias 4 -> 0
- net B: track 0.00 -> 98.7 mm, vias 0 -> 4
- net /B: track 98.7 -> 0.00 mm, vias 4 -> 0
- net /G: track 94.6 -> 0.00 mm, vias 4 -> 0
- net G: track 0.00 -> 94.6 mm, vias 0 -> 4
- net 3V8: track 15.5 -> 39.0 mm
- net /Microcontroller/SW2: track 0.00 -> 21.0 mm, vias 0 -> 3
- net /Microcontroller/SW3: track 0.00 -> 14.9 mm, vias 0 -> 1
- net /Microcontroller/SW1: track 0.00 -> 10.6 mm, vias 0 -> 1
- net Net-(C1-Pad2): track 10.4 -> 0.00 mm
- net +3V3: track 24.7 -> 32.7 mm, vias 5 -> 8
- net Net-(Q15-Pad3): track 0.00 -> 7.68 mm
- net Net-(Q15-Pad1): track 0.00 -> 6.33 mm
- net Net-(Q11-Pad2): track 0.00 -> 6.21 mm
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Other:
- board text added: "High-Power LED module - Rev0.4"
- board text removed: "High-Power Addressable LED module - Rev0.2"
