File: AddressableV3/AddressableLED.sch (KiCad schematic (older format))
At the start: 77 parts, among them J1 Conn_ARM_JTAG_SWD_10, J2 Conn_01x04_Female, J3 Conn_01x04_Female, Q1 MMBT3904, Q10 MMBT3904, Q11 DMN2041L, Q12 DMN2041L, Q13 DMN2041L, Q14 MMBT3904, Q15 MMBT3904, Q16 MMBT3904, Q17 DMN2041L, Q18 DMN2041L, Q19 DMN2041L, Q2 DMN2041L, Q20 MMBT3904, Q21 MMBT3904, Q22 MMBT3904, Q23 DMN2041L, Q24 DMN2041L, Q25 DMN2041L, Q3 MMBT3904, Q4 DMN2041L, Q5 MMBT3904, Q6 DMN2041L, Q7 MMBT3904, Q8 MMBT3904, Q9 MMBT3904, U1 STM32F030F4Px, U5 MCP1812AT-033_TT

Commit message: Desktop
Parts:
- removed R21, R22, R29: 22, Resistor_SMD:R_0603_1608Metric, symbol Device:R
Connections:
- net RESET: now also J1.10 (~RESET~)
- net SWCLK: now also J1.2 (SWDIO/TMS)
- net SWDIO: now also J1.4 (SWDCLK/TCK)
- removed net SCL: J2.4 (Pin_4), J3.4 (Pin_4), U1.17 (PA9)
- removed net SDA: J2.3 (Pin_3), J3.3 (Pin_3), U1.18 (PA10)
Changed lines of the file:
@@
 $EndComp
-Wire Wire Line
-	1500 2500 1700 2500
-Wire Wire Line
-	1500 2600 1700 2600
 Wire Wire Line
 	1500 2700 1700 2700
@@
 	0    -1   -1   0
 $EndComp
-Text Label 1700 2600 0    50   ~ 0
-SDA
-Text Label 1700 2500 0    50   ~ 0
-SCL
 $Comp
 L Connector:Conn_01x04_Female J3
@@
 $EndComp
 Wire Wire Line
-	17750 3000 17950 3000
-Wire Wire Line
-	17750 3100 17950 3100
-Wire Wire Line
 	17750 3200 17950 3200
 Wire Wire Line
@@
 	0    -1   -1   0
 $EndComp
-Text Label 17950 3100 0    50   ~ 0
-SDA
-Text Label 17950 3000 0    50   ~ 0
-SCL
 $Comp
 L power:+VDC #PWR0111
@@
 RESET
 $Comp
-L Device:R R29
-U 1 1 5E777D3A
-P 3350 4350
-F 0 "R29" V 3143 4350 50  0000 C CNN
-F 1 "22" V 3234 4350 50  0000 C CNN
-F 2 "Resistor_SMD:R_0603_1608Metric" V 3280 4350 50  0001 C CNN
-F 3 "~" H 3350 4350 50  0001 C CNN
-	1    3350 4350
-	0    -1   -1   0
-$EndComp
-Wire Wire Line
-	2400 4000 2700 4000
-Wire Wire Line
-	3000 4000 3700 4000
-Wire Wire Line
-	3500 4150 3700 4150
-$Comp
-L Device:R R22
-U 1 1 5E968443
-P 3350 4150
-F 0 "R22" V 3143 4150 50  0000 C CNN
-F 1 "22" V 3234 4150 50  0000 C CNN
-F 2 "Resistor_SMD:R_0603_1608Metric" V 3280 4150 50  0001 C CNN
-F 3 "~" H 3350 4150 50  0001 C CNN
-	1    3350 4150
-	0    1    1    0
-$EndComp
-$Comp
-L Device:R R21
-U 1 1 5E97F985
-P 2850 4000
-F 0 "R21" V 2643 4000 50  0000 C CNN
-F 1 "22" V 2734 4000 50  0000 C CNN
-F 2 "Resistor_SMD:R_0603_1608Metric" V 2780 4000 50  0001 C CNN
-F 3 "~" H 2850 4000 50  0001 C CNN
-	1    2850 4000
-	0    1    1    0
-$EndComp
-$Comp
 L power:GND #PWR0127
 U 1 1 5E9BA491
@@
 Wire Wire Line
 	3600 7300 4450 7300
-Wire Wire Line
-	3600 7400 3750 7400
-Wire Wire Line
-	3600 7500 3750 7500
-Text Label 3750 7400 0    50   ~ 0
-SCL
-Text Label 3750 7500 0    50   ~ 0
-SDA
 $Comp
 L Connector:Conn_ARM_JTAG_SWD_10 J1
@@
 	3000 4200 3000 4150
 Wire Wire Line
-	3000 4150 3200 4150
-Wire Wire Line
 	3000 4300 3000 4350
-Wire Wire Line
-	3000 4350 3200 4350
-Wire Wire Line
-	3500 4350 3700 4350
 $Comp
 L power:+3.3V #PWR0116
@@
 Wire Wire Line
 	15450 11050 15450 11450
+Wire Wire Line
+	2400 4000 3700 4000
+Wire Wire Line
+	3000 4150 3700 4150
+Wire Wire Line
+	3000 4350 3700 4350
 $EndSCHEMATC

Commit message: Desktop
Parts:
- removed J2: Conn_01x04_Female, AddressableLED:1.5mmHole, symbol Connector:Conn_01x04_Female
- removed J3: Conn_01x04_Female, AddressableLED:1.5mmHoleMirror, symbol Connector:Conn_01x04_Female
- removed Q7: MMBT3904, Package_TO_SOT_SMD:SOT-23, symbol Transistor_BJT:MMBT3904
- removed R10: 1k, Resistor_SMD:R_0603_1608Metric, symbol Device:R
- added H1, H2: MountingHole, MountingHole:MountingHole_3.2mm_M3, symbol Mechanical:MountingHole
- added J2, J3: Conn_01x02_Female, Connector_JST:JST_VH_B2P-VH_1x02_P3.96mm_Vertical, symbol Connector:Conn_01x02_Female
- added R21: 0, Resistor_SMD:R_0603_1608Metric, symbol Device:R
- added SW1, SW2, SW3: SW_DIP_x02, Logan:SideMountSwitch, symbol Switch:SW_DIP_x02
Connections:
- net +3V3: now also C2.1, U5.1 (3.3V)
- net +VDC: now also J2.1 (Pin_1), J3.1 (Pin_1)
- net GND: now also J2.2 (Pin_2), J3.2 (Pin_2)
- net RESET: now also R21.1; no longer J1.10 (~RESET~)
- net SWCLK: now also J1.4 (SWDCLK/TCK); no longer J1.2 (SWDIO/TMS)
- net SWDIO: now also J1.2 (SWDIO/TMS); no longer J1.4 (SWDCLK/TCK)
- new net: J1.10 (~RESET~), R21.2
Other:
- moved on the sheet: C2, D5, R30
Changed lines of the file:
@@
 L Device:C C2
 U 1 1 5DE90BBF
-P 3800 1900
-F 0 "C2" H 3915 1946 50  0000 L CNN
-F 1 "22u" H 3915 1855 50  0000 L CNN
-F 2 "Capacitor_SMD:C_0603_1608Metric" H 3838 1750 50  0001 C CNN
-F 3 "~" H 3800 1900 50  0001 C CNN
-	1    3800 1900
+P 3400 1900
+F 0 "C2" H 3515 1946 50  0000 L CNN
+F 1 "22u" H 3515 1855 50  0000 L CNN
+F 2 "Capacitor_SMD:C_0603_1608Metric" H 3438 1750 50  0001 C CNN
+F 3 "~" H 3400 1900 50  0001 C CNN
+	1    3400 1900
 	1    0    0    -1
 $EndComp
@@
 L power:+3.3V #PWR0108
 U 1 1 5DF45EC0
-P 4750 1150
-F 0 "#PWR0108" H 4750 1000 50  0001 C CNN
-F 1 "+3.3V" H 4765 1323 50  0000 C CNN
-F 2 "" H 4750 1150 50  0001 C CNN
-F 3 "" H 4750 1150 50  0001 C CNN
-	1    4750 1150
+P 3850 1550
+F 0 "#PWR0108" H 3850 1400 50  0001 C CNN
+F 1 "+3.3V" H 3865 1723 50  0000 C CNN
+F 2 "" H 3850 1550 50  0001 C CNN
+F 3 "" H 3850 1550 50  0001 C CNN
+	1    3850 1550
 	1    0    0    -1
 $EndComp
@@
 RESET
 Text Label 3700 4150 0    50   ~ 0
+SWCLK
+Text Label 3700 4350 0    50   ~ 0
 SWDIO
-Text Label 3700 4350 0    50   ~ 0
-SWCLK
 $Comp
 L power:GND #PWR0114
@@
 	1    0    0    -1
 $EndComp
-$Comp
-L Transistor_BJT:MMBT3904 Q7
-U 1 1 5E4A69EC
-P 4100 1350
-F 0 "Q7" H 4291 1396 50  0000 L CNN
-F 1 "MMBT3904" H 4291 1305 50  0000 L CNN
-F 2 "Package_TO_SOT_SMD:SOT-23" H 4300 1275 50  0001 L CIN
-F 3 "https://www.fairchildsemi.com/datasheets/2N/2N3904.pdf" H 4100 1350 50  0001 L CNN
-	1    4100 1350
-	0    -1   -1   0
-$EndComp
-Wire Wire Line
-	3150 1650 3250 1650
-$Comp
-L Device:R R10
-U 1 1 5E54B591
-P 3450 1650
-F 0 "R10" V 3243 1650 50  0000 C CNN
-F 1 "1k" V 3334 1650 50  0000 C CNN
-F 2 "Resistor_SMD:R_0603_1608Metric" V 3380 1650 50  0001 C CNN
-F 3 "~" H 3450 1650 50  0001 C CNN
-	1    3450 1650
-	0    1    1    0
-$EndComp
-Wire Wire Line
-	4100 1650 4100 1550
-Wire Wire Line
-	3600 1650 3800 1650
-Wire Wire Line
-	3800 1750 3800 1650
-Connection ~ 3800 1650
-Wire Wire Line
-	3800 1650 4100 1650
-Wire Wire Line
-	2800 2050 3800 2050
-Wire Wire Line
-	3250 1650 3250 1250
-Wire Wire Line
-	3250 1250 3900 1250
-Connection ~ 3250 1650
-Wire Wire Line
-	3250 1650 3300 1650
-Wire Wire Line
-	4300 1250 4750 1250
-Wire Wire Line
-	4750 1250 4750 1150
+Wire Wire Line
+	3400 1750 3400 1650
+Wire Wire Line
+	2800 2050 3400 2050
+Wire Wire Line
+	3400 1650 3850 1650
+Wire Wire Line
+	3850 1650 3850 1550
 $Comp
 L power:+3.3V #PWR0115
@@
 Wire Wire Line
 	7800 4750 7800 5050
-$Comp
-L Connector:Conn_01x04_Female J2
-U 1 1 5E781D58
-P 1300 2700
-F 0 "J2" H 1328 2676 50  0000 L CNN
-F 1 "Conn_01x04_Female" H 1328 2585 50  0000 L CNN
-F 2 "AddressableLED:1.5mmHole" H 1300 2700 50  0001 C CNN
-F 3 "~" H 1300 2700 50  0001 C CNN
-	1    1300 2700
-	-1   0    0    1
-$EndComp
 Wire Wire Line
 	1500 2700 1700 2700
@@
 	1    1700 2700
 	0    -1   -1   0
-$EndComp
-$Comp
-L Connector:Conn_01x04_Female J3
-U 1 1 5E87A062
-P 17550 3200
-F 0 "J3" H 17578 3176 50  0000 L CNN
-F 1 "Conn_01x04_Female" H 17578 3085 50  0000 L CNN
-F 2 "AddressableLED:1.5mmHoleMirror" H 17550 3200 50  0001 C CNN
-F 3 "~" H 17550 3200 50  0001 C CNN
-	1    17550 3200
-	-1   0    0    1
 $EndComp
 Wire Wire Line
@@
 L Device:LED D5
 U 1 1 5EDF6AE7
-P 5250 1250
-F 0 "D5" H 5243 995 50  0000 C CNN
-F 1 "LED" H 5243 1086 50  0000 C CNN
-F 2 "LED_SMD:LED_0603_1608Metric" H 5250 1250 50  0001 C CNN
-F 3 "~" H 5250 1250 50  0001 C CNN
-	1    5250 1250
+P 4350 1650
+F 0 "D5" H 4343 1395 50  0000 C CNN
+F 1 "LED" H 4343 1486 50  0000 C CNN
+F 2 "LED_SMD:LED_0603_1608Metric" H 4350 1650 50  0001 C CNN
+F 3 "~" H 4350 1650 50  0001 C CNN
+	1    4350 1650
 	-1   0    0    1
 $EndComp
 Wire Wire Line
-	4750 1250 5100 1250
-Connection ~ 4750 1250
+	3850 1650 4200 1650
+Connection ~ 3850 1650
 $Comp
 L Device:R R30
 U 1 1 5EE398AF
-P 5700 1500
-F 0 "R30" V 5493 1500 50  0000 C CNN
-F 1 "220" V 5584 1500 50  0000 C CNN
-F 2 "Resistor_SMD:R_0603_1608Metric" V 5630 1500 50  0001 C CNN
-F 3 "~" H 5700 1500 50  0001 C CNN
-	1    5700 1500
-	1    0    0    -1
-$EndComp
-Wire Wire Line
-	5400 1250 5700 1250
-Wire Wire Line
-	5700 1250 5700 1350
-Wire Wire Line
-	5700 1650 5700 1750
+P 4800 1900
+F 0 "R30" V 4593 1900 50  0000 C CNN
+F 1 "220" V 4684 1900 50  0000 C CNN
+F 2 "Resistor_SMD:R_0603_1608Metric" V 4730 1900 50  0001 C CNN
+F 3 "~" H 4800 1900 50  0001 C CNN
+	1    4800 1900
+	1    0    0    -1
+$EndComp
+Wire Wire Line
+	4500 1650 4800 1650
+Wire Wire Line
+	4800 1650 4800 1750
+Wire Wire Line
+	4800 2050 4800 2150
 $Comp
 L power:GND #PWR0134
 U 1 1 5EE60BC5
-P 5700 1750
-F 0 "#PWR0134" H 5700 1500 50  0001 C CNN
-F 1 "GND" H 5705 1577 50  0000 C CNN
-F 2 "" H 5700 1750 50  0001 C CNN
-F 3 "" H 5700 1750 50  0001 C CNN
-	1    5700 1750
+P 4800 2150
+F 0 "#PWR0134" H 4800 1900 50  0001 C CNN
+F 1 "GND" H 4805 1977 50  0000 C CNN
+F 2 "" H 4800 2150 50  0001 C CNN
+F 3 "" H 4800 2150 50  0001 C CNN
+	1    4800 2150
 	1    0    0    -1
 $EndComp
@@
 	15450 11050 15450 11450
 Wire Wire Line
-	2400 4000 3700 4000
+	2400 4000 2800 4000
 Wire Wire Line
 	3000 4150 3700 4150
 Wire Wire Line
 	3000 4350 3700 4350
+$Comp
+L Mechanical:MountingHole H1
+U 1 1 5EBB408E
+P 17275 6725
+F 0 "H1" H 17375 6771 50  0000 L CNN
+F 1 "MountingHole" H 17375 6680 50  0000 L CNN
+F 2 "MountingHole:MountingHole_3.2mm_M3" H 17275 6725 50  0001 C CNN
+F 3 "~" H 17275 6725 50  0001 C CNN
+	1    17275 6725
+	1    0    0    -1
+$EndComp
+$Comp
+L Mechanical:MountingHole H2
+U 1 1 5EBB5124
+P 17575 6725
+F 0 "H2" H 17675 6771 50  0000 L CNN
+F 1 "MountingHole" H 17675 6680 50  0000 L CNN
+F 2 "MountingHole:MountingHole_3.2mm_M3" H 17575 6725 50  0001 C CNN
+F 3 "~" H 17575 6725 50  0001 C CNN
+	1    17575 6725
+	1    0    0    -1
+$EndComp
+Wire Wire Line
+	3100 4000 3700 4000
+$Comp
+L Device:R R21
+U 1 1 5EC73DAD
+P 2950 4000
+F 0 "R21" V 2743 4000 50  0000 C CNN
+F 1 "0" V 2834 4000 50  0000 C CNN
+F 2 "Resistor_SMD:R_0603_1608Metric" V 2880 4000 50  0001 C CNN
+F 3 "~" H 2950 4000 50  0001 C CNN
+	1    2950 4000
+	0    1    1    0
+$EndComp
+Wire Wire Line
+	3150 1650 3400 1650
+Connection ~ 3400 1650
+$Comp
+L Connector:Conn_01x02_Female J2
+U 1 1 5EE42FDA
+P 1300 2800
+F 0 "J2" H 1192 2475 50  0000 C CNN
+F 1 "Conn_01x02_Female" H 1192 2566 50  0000 C CNN
+F 2 "Connector_JST:JST_VH_B2P-VH_1x02_P3.96mm_Vertical" H 1300 2800 50  0001 C CNN
+F 3 "~" H 1300 2800 50  0001 C CNN
+	1    1300 2800
+	-1   0    0    1
+$EndComp
+$Comp
+L Connector:Conn_01x02_Female J3
+U 1 1 5EE7B55E
+P 17550 3300
+F 0 "J3" H 17442 2975 50  0000 C CNN
+F 1 "Conn_01x02_Female" H 17442 3066 50  0000 C CNN
+F 2 "Connector_JST:JST_VH_B2P-VH_1x02_P3.96mm_Vertical" H 17550 3300 50  0001 C CNN
+F 3 "~" H 17550 3300 50  0001 C CNN
+	1    17550 3300
+	-1   0    0    1
+$EndComp
+$Comp
+L Switch:SW_DIP_x02 SW1
+U 1 1 5EE9C722
+P 17050 2550
+F 0 "SW1" H 17050 2917 50  0000 C CNN
+F 1 "SW_DIP_x02" H 17050 2826 50  0000 C CNN
+F 2 "Logan:SideMountSwitch" H 17050 2550 50  0001 C CNN
+F 3 "~" H 17050 2550 50  0001 C CNN
+	1    17050 2550
+	1    0    0    -1
+$EndComp
+$Comp
+L Switch:SW_DIP_x02 SW2
+U 1 1 5EED4A47
+P 17775 2550
+F 0 "SW2" H 17775 2917 50  0000 C CNN
+F 1 "SW_DIP_x02" H 17775 2826 50  0000 C CNN
+F 2 "Logan:SideMountSwitch" H 17775 2550 50  0001 C CNN
+F 3 "~" H 17775 2550 50  0001 C CNN
+	1    17775 2550
+	1    0    0    -1
+$EndComp
+$Comp
+L Switch:SW_DIP_x02 SW3
+U 1 1 5EEE6CA2
+P 18475 2550
+F 0 "SW3" H 18475 2917 50  0000 C CNN
+F 1 "SW_DIP_x02" H 18475 2826 50  0000 C CNN
+F 2 "Logan:SideMountSwitch" H 18475 2550 50  0001 C CNN
+F 3 "~" H 18475 2550 50  0001 C CNN
+	1    18475 2550
+	1    0    0    -1
+$EndComp
 $EndSCHEMATC

Commit message: Desktop
Parts:
- removed C1, C2: 22u, Capacitor_SMD:C_0603_1608Metric, symbol Device:C
- removed C4: 10u, Capacitor_SMD:C_0603_1608Metric, symbol Device:C
- removed C5: 100n, Capacitor_SMD:C_0603_1608Metric, symbol Device:C
- removed D5: LED, LED_SMD:LED_0603_1608Metric, symbol Device:LED
- removed J1: Conn_ARM_JTAG_SWD_10, Connector_PinHeader_1.27mm:PinHeader_2x05_P1.27mm_Vertical_SMD, symbol Connector:Conn_ARM_JTAG_SWD_10
- removed R21: 0, Resistor_SMD:R_0603_1608Metric, symbol Device:R
- removed R30: 220, Resistor_SMD:R_0603_1608Metric, symbol Device:R
- removed R9: 10k, Resistor_SMD:R_0603_1608Metric, symbol Device:R
- removed SW1, SW2, SW3: SW_DIP_x02, Logan:SideMountSwitch, symbol Switch:SW_DIP_x02
- removed U1: STM32F030F4Px, Package_SO:TSSOP-20_4.4x6.5mm_P0.65mm, symbol MCU_ST_STM32F0:STM32F030F4Px
- removed U5: MCP1812AT-033_TT, Package_TO_SOT_SMD:SOT-23, symbol AddressableLEDBJT:MCP1812AT-033_TT
- J2: footprint Connector_JST:JST_VH_B2P-VH_1x02_P3.96mm_Vertical -> AddressableLED:1.5mmHole
- J3: footprint Connector_JST:JST_VH_B2P-VH_1x02_P3.96mm_Vertical -> AddressableLED:1.5mmHoleMirror
Connections:
- net +VDC renamed 3V8
- net 3V8: no longer J2.1 (Pin_1), J3.1 (Pin_1)
- new net VDC: J2.1 (Pin_1), J3.1 (Pin_1)
Other:
- note removed: "Output = 2.7V with 1k Res"
- moved on the sheet: D1, D10, D11, D12, D13, D2, D3, D4, D6, D7, D8, D9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

Commit message: Desktop
Parts:
- removed J3: Conn_01x02_Female, AddressableLED:1.5mmHoleMirror, symbol Connector:Conn_01x02_Female
- added U1: LoganSWModule, Logan:Logan_SWmodule, symbol Logan:LoganSWModule
Connections:
- net 3V8: now also U1.5 (Vout), U1.6 (Vout)
- net GND: now also U1.1 (GND), U1.2 (GND), U1.7 (GND), U1.8 (GND)
- net VDC: now also U1.3 (Vin), U1.4 (Vin)
Changed lines of the file:
@@
-	0    -1   -1   0
-$EndComp
-Wire Wire Line
-	3650 1900 3850 1900
-Wire Wire Line
-	3650 2000 3850 2000
-$Comp
-L power:GND #PWR0125
-U 1 1 5E87A072
-P 3850 1900
-F 0 "#PWR0125" H 3850 1650 50  0001 C CNN
-F 1 "GND" V 3855 1772 50  0000 R CNN
-F 2 "" H 3850 1900 50  0001 C CNN
-F 3 "" H 3850 1900 50  0001 C CNN
-	1    3850 1900
 	0    -1   -1   0
 $EndComp
@@
 	-1   0    0    1
 $EndComp
-$Comp
-L Connector:Conn_01x02_Female J3
-U 1 1 5EE7B55E
-P 3450 2000
-F 0 "J3" H 3342 1675 50  0000 C CNN
-F 1 "Conn_01x02_Female" H 3342 1766 50  0000 C CNN
-F 2 "AddressableLED:1.5mmHoleMirror" H 3450 2000 50  0001 C CNN
-F 3 "~" H 3450 2000 50  0001 C CNN
-	1    3450 2000
-	-1   0    0    1
-$EndComp
 $Sheet
 S 5825 1275 2725 2025
@@
 	1    0    0    -1
 $EndComp
-Text Label 4825 13300 2    50   ~ 0
-B
 Wire Wire Line
 	5225 13300 4825 13300
@@
 	1    0    0    -1
 $EndComp
-Text Label 10675 13300 2    50   ~ 0
-R
 Wire Wire Line
 	11075 13300 10675 13300
@@
 	1    0    0    -1
 $EndComp
-Text Label 7825 13300 2    50   ~ 0
-G
 Wire Wire Line
 	8225 13300 7825 13300
@@
 	1    0    0    -1
 $EndComp
-Text Label 4825 10300 0    50   ~ 0
-B
 Wire Wire Line
 	5225 10300 4825 10300
@@
 	1    0    0    -1
 $EndComp
-Text Label 10675 10300 2    50   ~ 0
-R
 Wire Wire Line
 	11075 10300 10675 10300
@@
 	1    0    0    -1
 $EndComp
-Text Label 7825 10300 2    50   ~ 0
-G
 Wire Wire Line
 	8225 10300 7825 10300
@@
 	1    0    0    -1
 $EndComp
-Text Label 4825 7250 0    50   ~ 0
-B
 Wire Wire Line
 	5225 7250 4825 7250
@@
 	1    0    0    -1
 $EndComp
-Text Label 10675 7250 2    50   ~ 0
-R
 Wire Wire Line
 	11075 7250 10675 7250
@@
 	1    0    0    -1
 $EndComp
-Text Label 7825 7250 2    50   ~ 0
-G
 Wire Wire Line
 	8225 7250 7825 7250
@@
 	1    0    0    -1
 $EndComp
-Text Label 4825 4300 0    50   ~ 0
-B
 Wire Wire Line
 	5225 4300 4825 4300
@@
 	1    0    0    -1
 $EndComp
-Text Label 10675 4300 2    50   ~ 0
-R
 Wire Wire Line
 	11075 4300 10675 4300
@@
 	1    0    0    -1
 $EndComp
-Text Label 7825 4300 2    50   ~ 0
-G
 Wire Wire Line
 	8225 4300 7825 4300
@@
 Wire Wire Line
 	13075 13700 13075 14100
-Text GLabel 1450 3250 0    50   Input ~ 0
-GND
+Text GLabel 2750 2000 2    50   Input ~ 0
+VDC
+Text GLabel 2275 3100 0    50   Input ~ 0
+3V8
+Wire Wire Line
+	2275 3100 2375 3100
+Wire Wire Line
+	2375 3100 2375 3150
+Wire Wire Line
+	2375 3150 2525 3150
+Wire Wire Line
+	2525 3050 2375 3050
+Wire Wire Line
+	2375 3050 2375 3100
+Connection ~ 2375 3100
+$Comp
+L power:GND #PWR?
+U 1 1 5ED735F2
+P 3750 2800
+AR Path="/5F00043F/5ED735F2" Ref="#PWR?"  Part="1"
+AR Path="/5ED735F2" Ref="#PWR0111"  Part="1"
+F 0 "#PWR0111" H 3750 2550 50  0001 C CNN
+F 1 "GND" H 3755 2627 50  0000 C CNN
+F 2 "" H 3750 2800 50  0001 C CNN
+F 3 "" H 3750 2800 50  0001 C CNN
+	1    3750 2800
+	1    0    0    -1
+$EndComp
+Wire Wire Line
+	3525 2850 3625 2850
+Wire Wire Line
+	3625 2850 3625 2800
+Wire Wire Line
+	3625 2800 3750 2800
+Wire Wire Line
+	3525 2750 3625 2750
+Wire Wire Line
+	3625 2750 3625 2800
+Connection ~ 3625 2800
+Wire Wire Line
+	1800 3575 1800 3850
+Wire Wire Line
+	1700 3575 1800 3575
 $Comp
 L power:GND #PWR?
 U 1 1 5F218C55
-P 1550 3525
+P 1800 3850
 AR Path="/5F00043F/5F218C55" Ref="#PWR?"  Part="1"
 AR Path="/5F218C55" Ref="#PWR0107"  Part="1"
-F 0 "#PWR0107" H 1550 3275 50  0001 C CNN
-F 1 "GND" H 1555 3352 50  0000 C CNN
-F 2 "" H 1550 3525 50  0001 C CNN
-F 3 "" H 1550 3525 50  0001 C CNN
-	1    1550 3525
-	1    0    0    -1
-$EndComp
-Wire Wire Line
-	1450 3250 1550 3250
-Wire Wire Line
-	1550 3250 1550 3525
-Text GLabel 2750 2000 2    50   Input ~ 0
+F 0 "#PWR0107" H 1800 3600 50  0001 C CNN
+F 1 "GND" H 1805 3677 50  0000 C CNN
+F 2 "" H 1800 3850 50  0001 C CNN
+F 3 "" H 1800 3850 50  0001 C CNN
+	1    1800 3850
+	1    0    0    -1
+$EndComp
+Text GLabel 1700 3575 0    50   Input ~ 0
+GND
+$Comp
+L power:GND #PWR?
+U 1 1 5EF86E72
+P 2300 2800
+AR Path="/5F00043F/5EF86E72" Ref="#PWR?"  Part="1"
+AR Path="/5EF86E72" Ref="#PWR0108"  Part="1"
+F 0 "#PWR0108" H 2300 2550 50  0001 C CNN
+F 1 "GND" H 2305 2627 50  0000 C CNN
+F 2 "" H 2300 2800 50  0001 C CNN
+F 3 "" H 2300 2800 50  0001 C CNN
+	1    2300 2800
+	-1   0    0    1
+$EndComp
+Wire Wire Line
+	2525 2750 2425 2750
+Wire Wire Line
+	2425 2750 2425 2800
+Wire Wire Line
+	2425 2800 2300 2800
+Wire Wire Line
+	2525 2850 2425 2850
+Wire Wire Line
+	2425 2850 2425 2800
+Connection ~ 2425 2800
+Text GLabel 3750 3100 2    50   Input ~ 0
 VDC
-Text GLabel 3850 2000 2    50   Input ~ 0
-VDC
+Wire Wire Line
+	3525 3050 3625 3050
+Wire Wire Line
+	3625 3050 3625 3100
+Wire Wire Line
+	3625 3100 3750 3100
+Wire Wire Line
+	3525 3150 3625 3150
+Wire Wire Line
+	3625 3150 3625 3100
+Connection ~ 3625 3100
+$Comp
+L Logan:LoganSWModule U1
+U 1 1 5EFE3F02
+P 3025 2950
+F 0 "U1" H 3025 3375 50  0000 C CNN
+F 1 "LoganSWModule" H 3025 3284 50  0000 C CNN
+F 2 "Logan:Logan_SWmodule" H 3025 3250 50  0001 C CNN
+F 3 "" H 3025 3250 50  0001 C CNN
+	1    3025 2950
+	1    0    0    -1
+$EndComp
+Text GLabel 4825 4300 0    50   Input ~ 0
+B
+Text GLabel 4825 7250 0    50   Input ~ 0
+B
+Text GLabel 4825 10300 0    50   Input ~ 0
+B
+Text GLabel 4825 13300 0    50   Input ~ 0
+B
+Text GLabel 7825 4300 0    50   Input ~ 0
+G
+Text GLabel 7825 7250 0    50   Input ~ 0
+G
+Text GLabel 7825 10300 0    50   Input ~ 0
+G
+Text GLabel 7825 13300 0    50   Input ~ 0
+G
+Text GLabel 10675 4300 0    50   Input ~ 0
+R
+Text GLabel 10675 7250 0    50   Input ~ 0
+R
+Text GLabel 10675 10300 0    50   Input ~ 0
+R
+Text GLabel 10675 13300 0    50   Input ~ 0
+R
 $EndSCHEMATC
