File: AddressableV3/Micro.sch (KiCad schematic (older format))
At the start: 10 parts, among them J1 Conn_ARM_JTAG_SWD_10, SW1 SW_DIP_x02, SW2 SW_DIP_x02, SW3 SW_DIP_x02, U3 STM32F030F4Px

Commit message: Desktop
Parts:
- removed R31: R, symbol Device:R
- added R10, R21, R9: 10k, Resistor_SMD:R_0603_1608Metric, symbol Device:R
Connections:
- net +3V3: now also R10.1, R21.1, R9.1
- net GND: now also SW1.1, SW1.2, SW2.1, SW2.2, SW3.1, SW3.2
- net SW3: now reaches U3.17 (PA9)
- net SW3: now also SW3.3, SW3.4, R21.2
- net SW1: now reaches U3.18 (PA10)
- net SW1: now also SW1.3, SW1.4, R9.2
- net SW2: now reaches U3.2 (PF0)
- net SW2: now also SW2.3, SW2.4, R10.2
Other:
- moved on the sheet: SW1, SW2, SW3
