File: AddressableV3/PowerSheet.sch (KiCad schematic (older format))
At the start: 15 parts, among them U1 TPS563200, U2 MCP1812AT-033_TT

Commit message: Desktop
Parts:
- removed R9: 10k, Resistor_SMD:R_0603_1608Metric, symbol Device:R
Connections:
- net VDC: now also U1.5 (EN)
Changed lines of the file:
@@
 Wire Wire Line
 	3575 3000 3575 3050
-Wire Wire Line
-	3575 3050 3750 3050
-$Comp
-L Device:R R?
-U 1 1 5F183C96
-P 3900 3050
-AR Path="/5F183C96" Ref="R?"  Part="1"
-AR Path="/5EE32213/5F183C96" Ref="R9"  Part="1"
-F 0 "R9" V 3693 3050 50  0000 C CNN
-F 1 "10k" V 3784 3050 50  0000 C CNN
-F 2 "Resistor_SMD:R_0603_1608Metric" V 3830 3050 50  0001 C CNN
-F 3 "~" H 3900 3050 50  0001 C CNN
-	1    3900 3050
-	0    -1   -1   0
-$EndComp
-Wire Wire Line
-	4050 3050 4300 3050
 Text GLabel 1075 2600 0    50   Input ~ 0
 GND
@@
 	0    -1   -1   0
 $EndComp
+Wire Wire Line
+	3575 3050 4300 3050
 $EndSCHEMATC

Commit message: Desktop
Parts:
- removed C1: 0.1u, Capacitor_SMD:C_0603_1608Metric, symbol Device:C
- removed C6, C7, C8, C9: 22u, Capacitor_SMD:C_0603_1608Metric, symbol Device:C
- removed L1: 2.2u, Inductor_SMD:L_Coilcraft_XxL4020, symbol pspice:INDUCTOR
- removed R10: 10k, Resistor_SMD:R_0603_1608Metric, symbol Device:R
- removed R21: 36k, Resistor_SMD:R_0603_1608Metric, symbol Device:R
- removed U1: TPS563200, Package_TO_SOT_SMD:SOT-23-6, symbol Regulator_Switching:TPS563200
