File: ElectronicLoad/ElectronicLoad.sch (KiCad schematic (older format))
At the start: 16 parts, among them J1 AdafruitConverter, J2 Conn_01x04_Female, Q1 IRF540N, U1 AD8605, U2 MCP4821, U3 STM32G030C6T6, U4 MCP1812AT-033

Commit message: Desktop push
Parts:
- removed C2: 10u, symbol Device:CP
- removed Q1: IRF540N, Package_TO_SOT_THT:TO-220-3_Vertical, symbol Transistor_FET:IRF540N
- removed U2: MCP4821, Package_SO:MSOP-10-1EP_3x3mm_P0.5mm_EP1.68x1.88mm, symbol Logan:MCP4821
- added C2, C6: 1u, Capacitor_SMD:C_0603_1608Metric, symbol Device:C
- added C7: 1000u, Capacitor_SMD:CP_Elec_16x17.5, symbol Device:CP
- added J3: Conn_01x02_Female, symbol Connector:Conn_01x02_Female
- added J4, J5: Conn_01x02_Female, Connector_PinSocket_2.54mm:PinSocket_1x02_P2.54mm_Vertical, symbol Connector:Conn_01x02_Female
- added Q1: BUK9M12-60EX, Package_TO_SOT_THT:TO-220-3_Vertical, symbol Transistor_FET:BUK9M12-60EX
- added U2: MCP48CXBX1, Package_SO:MSOP-10-1EP_3x3mm_P0.5mm_EP1.68x1.88mm, symbol Logan:MCP48CXBX1
- C1: value CP -> 10u; footprint (none) -> Capacitor_SMD:CP_Elec_6.3x7.7
- C3: value C -> 0.1u; footprint (none) -> Capacitor_SMD:C_0603_1608Metric
- C4: value 100n -> 0.1u; footprint (none) -> Capacitor_SMD:C_0603_1608Metric
- C5: value CP -> 4.7u; footprint (none) -> Capacitor_SMD:CP_Elec_4x4.5
- R2: footprint (none) -> Resistor_SMD:R_0603_1608Metric
- R3: value 1k -> 10; footprint (none) -> Resistor_SMD:R_0603_1608Metric
- gave numbers to parts that had none: 1
Connections:
- wire segments 94 -> 106
Other:
- moved on the sheet: C1, C3, C5, PS1, R1, R2, R3, U1, U4

Commit message: Laptop Push
Parts:
- removed C1: 10u, Capacitor_SMD:CP_Elec_6.3x7.7, symbol Device:CP
- removed C2, C6: 1u, Capacitor_SMD:C_0603_1608Metric, symbol Device:C
- removed C3, C4: 0.1u, Capacitor_SMD:C_0603_1608Metric, symbol Device:C
- removed C5: 4.7u, Capacitor_SMD:CP_Elec_4x4.5, symbol Device:CP
- removed C7: 1000u, Capacitor_SMD:CP_Elec_16x17.5, symbol Device:CP
- removed J4, J5: Conn_01x02_Female, Connector_PinSocket_2.54mm:PinSocket_1x02_P2.54mm_Vertical, symbol Connector:Conn_01x02_Female
- removed PS1: IRM-02-5, Converter_ACDC:Converter_ACDC_MeanWell_IRM-02-xx_THT, symbol Converter_ACDC:IRM-02-5
- removed Q1: BUK9M12-60EX, Package_TO_SOT_THT:TO-220-3_Vertical, symbol Transistor_FET:BUK9M12-60EX
- removed R1: 0.1, Resistor_SMD:R_0603_1608Metric, symbol Device:R
- removed R2: 500, Resistor_SMD:R_0603_1608Metric, symbol Device:R
- removed R3: 10, Resistor_SMD:R_0603_1608Metric, symbol Device:R
- removed U1: AD8605, Package_TO_SOT_SMD:TSOT-23-5, symbol Logan:AD8605
- removed U2: MCP48CXBX1, Package_SO:MSOP-10-1EP_3x3mm_P0.5mm_EP1.68x1.88mm, symbol Logan:MCP48CXBX1
- removed U3: STM32G030C6T6, Package_QFP:LQFP-48_7x7mm_P0.5mm, symbol Logan:STM32G030C6T6
- removed U4: MCP1812AT-033, Package_TO_SOT_SMD:SOT-23, symbol Logan:MCP1812AT-033
Connections:
- net labels added: 3V3
- net labels removed: LINE, MISO, MOSI, NEUT, RESET, SCK, SWDCLK, SWDIO, VDC, ~CS, ~LAT
- wire segments 106 -> 31
Other:
- note removed: "CHECK POWER RAILS"
- moved on the sheet: J1, J3

Commit message: Desktop
Parts:
- removed J2: Conn_01x04_Female, symbol Connector:Conn_01x04_Female
- J3: footprint (none) -> Logan:5.7pitchHoles
Connections:
- net DC Driver/OUT+: now also J3.1 (Pin_1)
- net DC Driver/OUT-: now also J3.2 (Pin_2)
- net Microcontroller/RESET renamed Microcontroller/~RESET
Changed lines of the file:
@@
 EESchema Schematic File Version 4
 LIBS:ElectronicLoad-cache
-EELAYER 30 0
+EELAYER 29 0
 EELAYER END
 $Descr A4 11693 8268
@@
 	2575 4975 2575 5125
 $Comp
-L Connector:Conn_01x04_Female J2
-U 1 1 5EA9CC2A
-P 8950 1500
-F 0 "J2" H 8978 1476 50  0000 L CNN
-F 1 "Conn_01x04_Female" H 8978 1385 50  0000 L CNN
-F 2 "" H 8950 1500 50  0001 C CNN
-F 3 "~" H 8950 1500 50  0001 C CNN
-	1    8950 1500
-	-1   0    0    1
-$EndComp
-Wire Wire Line
-	9150 1300 9300 1300
-Wire Wire Line
-	9300 1300 9300 1200
-Wire Wire Line
-	9150 1500 9400 1500
-Wire Wire Line
-	9150 1600 9300 1600
-Wire Wire Line
-	9300 1600 9300 1700
-Wire Wire Line
-	9300 1700 9500 1700
-Text Label 9500 1550 0    50   ~ 0
-SCL
-Wire Wire Line
-	9400 1500 9400 1550
-Wire Wire Line
-	9400 1550 9500 1550
-Wire Wire Line
-	9150 1400 9400 1400
-Wire Wire Line
-	9400 1400 9400 1350
-Text Label 9500 1700 0    50   ~ 0
-SDA
-Wire Wire Line
-	9400 1350 9800 1350
-$Comp
 L Connector:Conn_01x02_Female J3
 U 1 1 5EA4144A
@@
 F 0 "J3" H 7803 4151 50  0000 L CNN
 F 1 "Conn_01x02_Female" H 7803 4060 50  0000 L CNN
-F 2 "" H 7775 4175 50  0001 C CNN
+F 2 "Logan:5.7pitchHoles" H 7775 4175 50  0001 C CNN
 F 3 "~" H 7775 4175 50  0001 C CNN
 	1    7775 4175
@@
 F1 "PowerSheet.sch" 50
 $EndSheet
-Text GLabel 9800 1200 2    50   Input ~ 0
-3V3
-Wire Wire Line
-	9300 1200 9800 1200
-Text GLabel 9800 1350 2    50   Input ~ 0
-GND
 Text GLabel 1000 1175 0    50   Input ~ 0
 3V3
@@
 	1175 1325 1175 1350
 $Sheet
-S 3975 3725 1275 1150
+S 3975 3700 1275 1150
 U 5EDE0641
 F0 "Microcontroller" 50
 F1 "Mirco.sch" 50
-F2 "RESET" I L 3975 4075 50
-F3 "~LAT" I R 5250 3875 50
-F4 "SCK" I R 5250 3975 50
-F5 "~CS" I R 5250 4075 50
-F6 "MOSI" I R 5250 4175 50
-F7 "MISO" I R 5250 4275 50
-F8 "SCL" I R 5250 4675 50
-F9 "SDA" I R 5250 4775 50
-F10 "SWDIO" I L 3975 4275 50
-F11 "SWCLK" I L 3975 4375 50
+F2 "~LAT" I R 5250 3850 50
+F3 "SCK" I R 5250 3950 50
+F4 "~CS" I R 5250 4050 50
+F5 "MOSI" I R 5250 4150 50
+F6 "MISO" I R 5250 4250 50
+F7 "SCL" I R 5250 4650 50
+F8 "SDA" I R 5250 4750 50
+F9 "SWDIO" I L 3975 4275 50
+F10 "SWCLK" I L 3975 4375 50
+F11 "~RESET" I L 3975 4075 50
+F12 "ADC_in0" I R 5250 4500 50
 $EndSheet
-Wire Wire Line
-	5250 3875 5625 3875
-Wire Wire Line
-	5250 3975 5625 3975
-Wire Wire Line
-	5250 4075 5625 4075
-Wire Wire Line
-	5250 4175 5625 4175
-Wire Wire Line
-	5250 4275 5625 4275
 $Comp
 L power:+3V3 #PWR0103
@@
 	3075 4375 3975 4375
 $Sheet
-S 5625 3725 1150 1150
+S 5650 3700 1150 1150
 U 5EC9D635
 F0 "DC Driver" 50
 F1 "DCDriverSheet.sch" 50
-F2 "OUT+" I R 6775 4000 50
-F3 "OUT-" I R 6775 4500 50
-F4 "~LAT" I L 5625 3875 50
-F5 "SCK" I L 5625 3975 50
-F6 "~CS" I L 5625 4075 50
-F7 "MOSI" I L 5625 4175 50
-F8 "MISO" I L 5625 4275 50
-F9 "I_SENSE" I L 5625 4550 50
+F2 "OUT+" I R 6800 3975 50
+F3 "OUT-" I R 6800 4475 50
+F4 "~LAT" I L 5650 3850 50
+F5 "SCK" I L 5650 3950 50
+F6 "~CS" I L 5650 4050 50
+F7 "MOSI" I L 5650 4150 50
+F8 "MISO" I L 5650 4250 50
+F9 "I_SENSE" I L 5650 4500 50
 $EndSheet
 $Sheet
@@
 F0 "LCD" 50
 F1 "LCD.sch" 50
-F2 "SCL" I L 5625 5675 50
+F2 "SCL" I L 5625 5600 50
 F3 "SDA" I L 5625 5775 50
 $EndSheet
 Wire Wire Line
-	5250 4675 5475 4675
+	5400 5775 5625 5775
 Wire Wire Line
-	5475 4675 5475 5675
+	5650 3850 5250 3850
 Wire Wire Line
-	5475 5675 5625 5675
+	5250 3950 5650 3950
 Wire Wire Line
-	5250 4775 5400 4775
+	5650 4050 5250 4050
 Wire Wire Line
-	5400 4775 5400 5775
+	5250 4150 5650 4150
 Wire Wire Line
-	5400 5775 5625 5775
+	5650 4250 5250 4250
+Wire Wire Line
+	5400 4750 5250 4750
+Wire Wire Line
+	5400 4750 5400 5775
+Wire Wire Line
+	5525 5600 5625 5600
+Wire Wire Line
+	5525 4650 5250 4650
+Wire Wire Line
+	5525 4650 5525 5600
+Wire Wire Line
+	6800 3975 7200 3975
+Wire Wire Line
+	7200 3975 7200 4175
+Wire Wire Line
+	7200 4175 7575 4175
+Wire Wire Line
+	6800 4475 7200 4475
+Wire Wire Line
+	7200 4475 7200 4275
+Wire Wire Line
+	7200 4275 7575 4275
+Wire Wire Line
+	5650 4500 5250 4500
 $EndSCHEMATC

Commit message: Desktop
Changed lines of the file:
@@
 F5 "MOSI" I R 5250 4150 50
 F6 "MISO" I R 5250 4250 50
-F7 "SCL" I R 5250 4650 50
-F8 "SDA" I R 5250 4750 50
-F9 "SWDIO" I L 3975 4275 50
-F10 "SWCLK" I L 3975 4375 50
-F11 "~RESET" I L 3975 4075 50
-F12 "ADC_in0" I R 5250 4500 50
+F7 "SWDIO" I L 3975 4275 50
+F8 "SWCLK" I L 3975 4375 50
+F9 "~RESET" I L 3975 4075 50
+F10 "ADC_in0" I R 5250 4500 50
+F11 "Data" I R 5250 4625 50
+F12 "EN" I R 5250 4700 50
+F13 "CLK" I R 5250 4775 50
 $EndSheet
 $Comp
@@
 F0 "LCD" 50
 F1 "LCD.sch" 50
-F2 "SCL" I L 5625 5600 50
-F3 "SDA" I L 5625 5775 50
+F2 "Data" I L 5625 5875 50
+F3 "CLK" I L 5625 6075 50
+F4 "EN" I L 5625 5975 50
 $EndSheet
-Wire Wire Line
-	5400 5775 5625 5775
 Wire Wire Line
 	5650 3850 5250 3850
@@
 Wire Wire Line
 	5650 4250 5250 4250
-Wire Wire Line
-	5400 4750 5250 4750
-Wire Wire Line
-	5400 4750 5400 5775
-Wire Wire Line
-	5525 5600 5625 5600
-Wire Wire Line
-	5525 4650 5250 4650
-Wire Wire Line
-	5525 4650 5525 5600
 Wire Wire Line
 	6800 3975 7200 3975
@@
 Wire Wire Line
 	5650 4500 5250 4500
+Wire Wire Line
+	5250 4775 5375 4775
+Wire Wire Line
+	5375 4775 5375 6075
+Wire Wire Line
+	5250 4700 5425 4700
+Wire Wire Line
+	5425 4700 5425 5975
+Wire Wire Line
+	5250 4625 5475 4625
+Wire Wire Line
+	5475 4625 5475 5875
+Wire Wire Line
+	5625 6075 5375 6075
+Wire Wire Line
+	5425 5975 5625 5975
+Wire Wire Line
+	5475 5875 5625 5875
 $EndSCHEMATC

Commit message: Laptop
Connections:
- net GND: now also J1.9 (GNDDetect)
Changed lines of the file:
@@
 EESchema Schematic File Version 4
 LIBS:ElectronicLoad-cache
-EELAYER 29 0
+EELAYER 30 0
 EELAYER END
 $Descr A4 11693 8268
@@
 	2575 3775 2575 3675
 Wire Wire Line
-	2575 4975 2575 5125
+	2575 4975 2575 5075
 $Comp
 L Connector:Conn_01x02_Female J3
@@
 Wire Wire Line
 	5475 5875 5625 5875
+Wire Wire Line
+	2575 5075 2475 5075
+Wire Wire Line
+	2475 5075 2475 4975
+Connection ~ 2575 5075
+Wire Wire Line
+	2575 5075 2575 5125
 $EndSCHEMATC
