File: ElectronicLoad/LCD.sch (KiCad schematic (older format))
At the start: 3 parts, among them J6 Conn_01x04_Female

Commit message: Desktop
Parts:
- removed J6: Conn_01x04_Female, Connector_PinHeader_2.54mm:PinHeader_1x04_P2.54mm_Vertical, symbol Connector:Conn_01x04_Female
- removed TP14, TP15: TestPoint, TestPoint:TestPoint_THTPad_D1.5mm_Drill0.7mm, symbol Connector:TestPoint
- added DS1: WC1602A, Connector_PinHeader_2.54mm:PinHeader_1x16_P2.54mm_Vertical, symbol Display_Character:WC1602A
- added R11: 220, Resistor_SMD:R_0603_1608Metric, symbol Device:R
- added RV1: R_POT, Logan:Potentiometer_Bourns_TC33X-2, symbol Device:R_POT
- added U7: 74HC595D, Package_SO:SOIC-16_3.9x9.9mm_P1.27mm, symbol Logan:74HC595D
Connections:
- net GND: now also DS1.1 (VSS), DS1.10 (D3), DS1.16 (LED(-)), DS1.5 (R/W), DS1.7 (D0), DS1.8 (D1), DS1.9 (D2), RV1.3, U7.13 (~OE), U7.8 (GND)
- new net: DS1.15 (LED(+)), R11.1
- new net: DS1.3 (VO), RV1.2
- new net: DS1.4 (RS), U7.4 (Q4)
- new net +5V: DS1.2 (VDD), R11.2, RV1.1, U7.10 (~MR), U7.16 (VCC)
- new net CLK: U7.11 (SHCP), U7.12 (STCP)
- new net D4: DS1.11 (D4), U7.15 (Q0)
- new net D5: DS1.12 (D5), U7.1 (Q1)
- new net D6: DS1.13 (D6), U7.2 (Q2)
- new net D7: DS1.14 (D7), U7.3 (Q3)
- new net Data: U7.14 (SER)
- new net EN: DS1.6 (E)
