File: ElectronicLoad/ElectronicLoad.kicad_pcb (KiCad board)
At the start: 2 copper layers, 5 parts, among them Q1 IRF540N, U1 AD8605, U2 MCP4821, U3 STM32F030F4Px

Commit message: push from desktop
Parts:
- added J1: AdafruitConverter, Connector_PinHeader_1.27mm:PinHeader_2x05_P1.27mm_Vertical_SMD, F.Cu at (179.8, 73.5)
- added PS1: IRM-02-3.3, Converter_ACDC:Converter_ACDC_MeanWell_IRM-02-xx_THT, F.Cu at (129.1, 46.0)
- added U3: STM32G030C6T6, Package_QFP:LQFP-48_7x7mm_P0.5mm, F.Cu at (180.7, 63.6)
- added U4: MCP1812AT-033, Package_TO_SOT_SMD:SOT-23, F.Cu at (177.2, 80.0)
- R1: value 5 -> 0.1
Connections:
- U1 pad 1: Net-(Q1-Pad1) -> Net-(R3-Pad2)
- U1 pad 2: Net-(U1-Pad2) -> GND
- U1 pad 4: Net-(Q1-Pad3) -> Net-(R2-Pad2)
- U1 pad 5: Net-(U1-Pad5) -> +3V3
- U2 pad 1: Net-(U2-Pad1) -> +3V3
- U2 pad 10: Net-(U2-Pad10) -> /MOSI
- U2 pad 2: Net-(U2-Pad2) -> /~CS
- U2 pad 6: Net-(U2-Pad6) -> /~LAT
- U2 pad 7: Net-(U2-Pad7) -> GND
- U2 pad 8: Net-(U2-Pad8) -> /MISO
- U2 pad 9: Net-(U2-Pad9) -> /SCK

Commit message: Desktop push
Parts:
- removed the U3 at (180.7, 63.6)
- removed the U3 at (162.3, 76.1)
- added C1: 10u, Capacitor_SMD:CP_Elec_6.3x7.7, F.Cu at (97.1, 55.5)
- added C2: 1u, Capacitor_SMD:C_0603_1608Metric, F.Cu at (78.1, 71.4)
- added C3: 0.1u, Capacitor_SMD:C_0603_1608Metric, F.Cu at (81.6, 71.4)
- added C4: 0.1u, Capacitor_SMD:C_0603_1608Metric, F.Cu at (86.1, 79.2)
- added C5: 4.7u, Capacitor_SMD:CP_Elec_4x4.5, F.Cu at (103.4, 45.5)
- added C6: 1u, Capacitor_SMD:C_0603_1608Metric, F.Cu at (101.3, 80.8)
- added C7: 1000u, Capacitor_SMD:CP_Elec_16x17.5, F.Cu at (81.8, 50.7)
- added J4: Conn_01x02_Female, Connector_PinSocket_2.54mm:PinSocket_1x02_P2.54mm_Vertical, F.Cu at (32.4, 43.3)
- added J5: Conn_01x02_Female, Connector_PinSocket_2.54mm:PinSocket_1x02_P2.54mm_Vertical, F.Cu at (82.2, 33.2)
- added R2: 500, Resistor_SMD:R_0603_1608Metric, F.Cu at (111.5, 64.0)
- added R3: 10, Resistor_SMD:R_0603_1608Metric, F.Cu at (108.6, 59.5)
- added U3: STM32G030C6T6, Package_QFP:LQFP-48_7x7mm_P0.5mm, F.Cu at (88.2, 70.4)
- PS1: value IRM-02-3.3 -> IRM-02-5
- Q1: value IRF540N -> BUK9M12-60EX
- U2: value MCP4821 -> MCP48CXBX1
- moved J1 119.5 mm to (60.5, 66.2)
- moved U4 89.1 mm to (95.2, 45.2)
- moved PS1 88.6 mm to (41.0, 36.3)
- moved U1 55.0 mm to (104.7, 63.3)
- moved U2 49.0 mm to (101.9, 70.9)
- moved Q1 37.1 mm to (119.9, 53.6), turned to 270 degrees
- moved R1 33.5 mm to (117.7, 70.2), turned to 270 degrees
Connections:
- Q1 pad 2: Net-(Q1-Pad2) -> Net-(Q1-Pad1)
- Q1 pad 3: Net-(Q1-Pad3) -> Net-(Q1-Pad1)
- R1 pad 1: Net-(Q1-Pad3) -> Net-(Q1-Pad1)

Commit message: Laptop Push
Parts:
- removed R2: 500, Resistor_SMD:R_0603_1608Metric
- added C10: 1u, Capacitor_SMD:C_0603_1608Metric, F.Cu at (169.2, 69.1)
- added C8: 1u, Capacitor_SMD:C_0603_1608Metric, F.Cu at (172.8, 62.1)
- added C9: 1u, Capacitor_SMD:C_0603_1608Metric, F.Cu at (176.8, 62.1)
- added F1: Fuse, Logan:FuseHolder5x20, F.Cu at (102.0, 87.8)
- added R4: 0.02, Resistor_SMD:R_0603_1608Metric, F.Cu at (168.5, 66.5)
- added R5: 0.02, Resistor_SMD:R_0603_1608Metric, F.Cu at (165.2, 70.0)
- added R7: 1k, Resistor_SMD:R_0603_1608Metric, F.Cu at (168.5, 64.0)
- added R8: 10k, Resistor_SMD:R_0603_1608Metric, F.Cu at (172.8, 59.6)
- added U5: AD8605, Package_TO_SOT_SMD:TSOT-23-5, F.Cu at (156.5, 71.1)
- added U6: AD8605, Package_TO_SOT_SMD:TSOT-23-5, F.Cu at (168.1, 60.6)
- C1: value 10u -> 1000u; footprint Capacitor_SMD:CP_Elec_6.3x7.7 -> Capacitor_SMD:CP_Elec_16x17.5
- C2: value 1u -> 10u; footprint Capacitor_SMD:C_0603_1608Metric -> Capacitor_SMD:CP_Elec_6.3x7.7
- C4: value 0.1u -> 4.7u; footprint Capacitor_SMD:C_0603_1608Metric -> Capacitor_SMD:CP_Elec_4x4.5
- C5: value 4.7u -> 1u; footprint Capacitor_SMD:CP_Elec_4x4.5 -> Capacitor_SMD:C_0603_1608Metric
- C6: value 1u -> 0.1u
- C7: value 1000u -> 1u; footprint Capacitor_SMD:CP_Elec_16x17.5 -> Capacitor_SMD:C_0603_1608Metric
- J5: footprint Connector_PinSocket_2.54mm:PinSocket_1x02_P2.54mm_Vertical -> Logan:16GAWire1x02
- Q1: value BUK9M12-60EX -> BUK9515-60E
- R1: value 0.1 -> 10
- R3: value 10 -> 1k
- U1: value AD8605 -> MCP1812AT-033; footprint Package_TO_SOT_SMD:TSOT-23-5 -> Package_TO_SOT_SMD:SOT-23
- U2: value MCP48CXBX1 -> STM32G030C6T6; footprint Package_SO:MSOP-10-1EP_3x3mm_P0.5mm_EP1.68x1.88mm -> Package_QFP:LQFP-48_7x7mm_P0.5mm
- U3: value STM32G030C6T6 -> MCP48CXBX1; footprint Package_QFP:LQFP-48_7x7mm_P0.5mm -> Package_SO:MSOP-10-1EP_3x3mm_P0.5mm_EP1.68x1.88mm
- U4: value MCP1812AT-033 -> AD8605; footprint Package_TO_SOT_SMD:SOT-23 -> Package_TO_SOT_SMD:TSOT-23-5
- moved J4 117.2 mm to (148.3, 60.7)
- moved J1 99.2 mm to (158.7, 80.6)
- moved C7 91.8 mm to (172.5, 64.6), turned to 0 degrees
- moved U4 71.9 mm to (163.8, 66.5)
- moved U3 69.4 mm to (157.5, 66.6), turned to 0 degrees
- moved J5 64.9 mm to (120.7, 85.4), turned to 0 degrees
- moved R1 60.0 mm to (176.8, 59.6), turned to 0 degrees
- moved PS1 57.7 mm to (92.3, 62.8)
- moved C3 57.2 mm to (138.4, 77.7), turned to 0 degrees
- moved C2 53.9 mm to (131.2, 80.6), turned to 0 degrees
- moved R3 53.7 mm to (161.2, 70.1), turned to 0 degrees
- moved C5 52.0 mm to (102.0, 97.6), turned to 0 degrees
- moved C4 44.5 mm to (129.9, 87.6)
- moved C1 39.9 mm to (135.1, 67.4), turned to 0 degrees
- moved Q1 38.1 mm to (157.1, 62.3), turned to 0 degrees
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Connections:
- C1 pad 1: VDC -> +5V
- C2 pad 1: +3V3 -> +5V
- C3 pad 1: VDC -> +5V
- C4 pad 1: +3V3 -> 3V3
- C5 pad 1: +3V3 -> 3V3
- C6 pad 1: +3V3 -> 3V3
- C7 pad 1: VDC -> +5V
- J1 pad 1: +3V3 -> 3V3
- J1 pad 10: /RESET -> Net-(J1-Pad10)
- J1 pad 2: /SWDCLK -> /Microcontroller/SWCLK
- J1 pad 4: /SWDIO -> /Microcontroller/SWDIO
- J4 pad 1: NEUT -> GND
- J4 pad 2: LINE -> +5V
- J5 pad 1: GND -> NEUT
- J5 pad 2: VDC -> Net-(F1-Pad2)
- PS1 pad 4: VDC -> +5V
- Q1 pad 2: Net-(Q1-Pad1) -> /DC Driver/OUT+
- Q1 pad 3: Net-(Q1-Pad1) -> Net-(Q1-Pad2)
- R1 pad 2: GND -> Net-(R1-Pad2)
- R3 pad 1: Net-(Q1-Pad4) -> Net-(Q1-Pad2)
- U1 pad 1: Net-(R3-Pad2) -> 3V3
- U1 pad 2: GND -> +5V
- U1 pad 3: Net-(U1-Pad3) -> GND
- U2 pad 1: +3V3 -> Net-(U2-Pad1)
- U2 pad 10: /MOSI -> /Microcontroller/~RESET
- U2 pad 11: (no net) -> Net-(U2-Pad11)
- U2 pad 2: /~CS -> Net-(U2-Pad2)
- U2 pad 4: Net-(U1-Pad3) -> 3V3
- U2 pad 6: /~LAT -> 3V3
- U2 pad 8: /MISO -> Net-(U2-Pad8)
- U2 pad 9: /SCK -> Net-(U2-Pad9)
- U3 pad 1: Net-(U3-Pad1) -> +5V
- U3 pad 10: /RESET -> /DC Driver/MOSI
- U3 pad 11: Net-(U3-Pad11) -> (no net)
- U3 pad 2: Net-(U3-Pad2) -> /DC Driver/~CS
- U3 pad 4: +3V3 -> Net-(U3-Pad4)
- U3 pad 6: +3V3 -> /DC Driver/~LAT
- U3 pad 8: Net-(U3-Pad8) -> /DC Driver/MISO
- U3 pad 9: Net-(U3-Pad9) -> /DC Driver/SCK
- U4 pad 1: +3V3 -> Net-(R1-Pad2)
- U4 pad 2: VDC -> GND
- U4 pad 3: GND -> Net-(U3-Pad4)

Commit message: Desktop
Parts:
- added C11: 8p, Capacitor_SMD:C_0603_1608Metric, F.Cu at (32.0, 96.0)
- added C12: 8p, Capacitor_SMD:C_0603_1608Metric, F.Cu at (40.0, 94.0)
- added C13: 1u, Capacitor_SMD:C_0603_1608Metric, F.Cu at (58.0, 89.0)
- added D1: LEDGREEN, LED_SMD:LED_0603_1608Metric, F.Cu at (30.0, 73.0)
- added J3: Conn_01x02_Female, Logan:5.7pitchHoles, F.Cu at (97.0, 85.0)
- added J6: Conn_01x04_Female, Connector_PinHeader_2.54mm:PinHeader_1x04_P2.54mm_Vertical, F.Cu at (39.0, 105.0)
- added R10: 1k, Resistor_SMD:R_0603_1608Metric, F.Cu at (63.0, 80.2)
- added R2: 1k, Resistor_SMD:R_0603_1608Metric, F.Cu at (66.8, 81.0)
- added R6: 100, Resistor_SMD:R_0603_1608Metric, F.Cu at (59.0, 92.0)
- added R9: 2k, Resistor_SMD:R_0603_1608Metric, F.Cu at (30.0, 77.0)
- added TP1: TestPoint, TestPoint:TestPoint_Pad_D2.0mm, F.Cu at (51.0, 70.6)
- added TP10: TestPoint, TestPoint:TestPoint_THTPad_D1.5mm_Drill0.7mm, F.Cu at (54.8, 101.2)
- added TP11: TestPoint, TestPoint:TestPoint_THTPad_D1.5mm_Drill0.7mm, F.Cu at (58.3, 97.7)
- added TP12: TestPoint, TestPoint:TestPoint_THTPad_D1.5mm_Drill0.7mm, F.Cu at (58.3, 101.2)
- added TP13: TestPoint, TestPoint:TestPoint_THTPad_D1.5mm_Drill0.7mm, F.Cu at (61.9, 97.7)
- added TP14: TestPoint, TestPoint:TestPoint_THTPad_D1.5mm_Drill0.7mm, F.Cu at (54.8, 104.9)
- added TP15: TestPoint, TestPoint:TestPoint_THTPad_D1.5mm_Drill0.7mm, F.Cu at (58.3, 104.9)
- added TP2: TestPoint, TestPoint:TestPoint_Pad_D2.0mm, F.Cu at (20.0, 45.0)
- added TP3: TestPoint, TestPoint:TestPoint_Pad_D2.0mm, F.Cu at (58.0, 72.0)
- added TP4: TestPoint, TestPoint:TestPoint_THTPad_D1.5mm_Drill0.7mm, F.Cu at (61.6, 101.7)
- added TP5: TestPoint, TestPoint:TestPoint_THTPad_D1.5mm_Drill0.7mm, F.Cu at (61.6, 105.2)
- added TP6: TestPoint, TestPoint:TestPoint_THTPad_D1.5mm_Drill0.7mm, F.Cu at (65.1, 101.7)
- added TP7: TestPoint, TestPoint:TestPoint_THTPad_D1.5mm_Drill0.7mm, F.Cu at (65.1, 105.2)
- added TP8: TestPoint, TestPoint:TestPoint_THTPad_D1.5mm_Drill0.7mm, F.Cu at (26.0, 103.0)
- added TP9: TestPoint, TestPoint:TestPoint_THTPad_D1.5mm_Drill0.7mm, F.Cu at (46.0, 99.0)
- added Y1: Crystal_GND24, Crystal:Crystal_SMD_3225-4Pin_3.2x2.5mm, F.Cu at (36.0, 94.0)
- R4, R5: footprint Resistor_SMD:R_0603_1608Metric -> Resistor_SMD:R_2512_6332Metric
- moved J1 130.8 mm to (27.9, 84.7)
- moved U6 119.3 mm to (52.0, 88.0)
- moved C10 115.4 mm to (55.0, 85.0)
- moved C7 114.0 mm to (60.0, 83.0), turned to 270 degrees
- moved C9 113.9 mm to (68.0, 96.0)
- moved R8 106.6 mm to (70.0, 88.0), turned to 180 degrees
- moved R1 105.3 mm to (73.0, 77.2), turned to 180 degrees
- moved J5 104.9 mm to (20.4, 54.5), turned to 270 degrees
- moved C8 104.6 mm to (69.0, 75.0), turned to 90 degrees
- moved R7 101.4 mm to (72.0, 95.0), turned to 90 degrees
- moved U3 100.4 mm to (57.9, 79.0), turned to 180 degrees
- moved U4 98.4 mm to (66.0, 77.0)
- moved R4 92.8 mm to (79.0, 91.0), turned to 270 degrees
- moved R3 89.0 mm to (74.0, 88.0), turned to 180 degrees
- moved U5 88.8 mm to (70.0, 91.0)
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Connections:
- C10 pad 1: 3V3 -> +5V
- C9 pad 1: 3V3 -> +5V
- J1 pad 10: Net-(J1-Pad10) -> /Microcontroller/~RESET
- U2 pad 11: Net-(U2-Pad11) -> /Microcontroller/ADC_in0
- U2 pad 8: Net-(U2-Pad8) -> /Microcontroller/12MHz_in
- U2 pad 9: Net-(U2-Pad9) -> /Microcontroller/12MHz_out
- U3 pad 4: Net-(U3-Pad4) -> Net-(C13-Pad1)
- U4 pad 3: Net-(U3-Pad4) -> Net-(R10-Pad1)
- U6 pad 1: /DC Driver/I_SENSE -> /Microcontroller/ADC_in0
- U6 pad 4: /DC Driver/I_SENSE -> /Microcontroller/ADC_in0

Commit message: Desktop
Parts:
- added DS1: WC1602A, Connector_PinHeader_2.54mm:PinHeader_1x16_P2.54mm_Vertical, F.Cu at (36.8, 122.2)
- added Q2: MMBT3904, Package_TO_SOT_SMD:SOT-23, F.Cu at (34.9, 71.5)
- added R11: 220, Resistor_SMD:R_0603_1608Metric, F.Cu at (63.8, 58.5)
- added RV1: R_POT, Logan:Potentiometer_Bourns_TC33X-2, F.Cu at (85.2, 190.8)
- added U7: 74HC595D, Package_SO:SOIC-16_3.9x9.9mm_P1.27mm, F.Cu at (53.9, 115.0)
Connections:
- U2 pad 29: /LCD/SCL -> /LCD/Data
- U2 pad 30: Net-(U2-Pad30) -> /LCD/CLK
- U2 pad 31: Net-(U2-Pad31) -> /LCD/EN
- U2 pad 32: /LCD/SDA -> Net-(U2-Pad32)
Routing:
- net LINE: track 0.00 -> 22.1 mm
- net Net-(F1-Pad2): track 0.00 -> 14.0 mm

Commit message: Laptop
Parts:
- removed C8: 1u, Capacitor_SMD:C_0603_1608Metric
- removed J6: Conn_01x04_Female, Connector_PinHeader_2.54mm:PinHeader_1x04_P2.54mm_Vertical
- removed TP14, TP15, TP6: TestPoint, TestPoint:TestPoint_THTPad_D1.5mm_Drill0.7mm
- added REF**: VIA-0.6mm, Logan:VIA-0.6mm, F.Cu at (21.8, 83.5)
- added REF**: VIA-0.6mm, Logan:VIA-0.6mm, F.Cu at (17.8, 82.5)
- added REF**: VIA-0.6mm, Logan:VIA-0.6mm, F.Cu at (21.8, 81.5)
- added REF**: VIA-0.6mm, Logan:VIA-0.6mm, F.Cu at (20.8, 81.5)
- added REF**: VIA-0.6mm, Logan:VIA-0.6mm, F.Cu at (19.8, 81.5)
- added REF**: VIA-0.6mm, Logan:VIA-0.6mm, F.Cu at (18.8, 81.5)
- added REF**: VIA-0.6mm, Logan:VIA-0.6mm, F.Cu at (17.8, 81.5)
- added REF**: VIA-0.6mm, Logan:VIA-0.6mm, F.Cu at (21.8, 80.5)
- added REF**: VIA-0.6mm, Logan:VIA-0.6mm, F.Cu at (20.8, 80.5)
- added REF**: VIA-0.6mm, Logan:VIA-0.6mm, F.Cu at (19.8, 80.5)
- added REF**: VIA-0.6mm, Logan:VIA-0.6mm, F.Cu at (18.8, 80.5)
- added REF**: VIA-0.6mm, Logan:VIA-0.6mm, F.Cu at (20.8, 83.5)
- added REF**: VIA-0.6mm, Logan:VIA-0.6mm, F.Cu at (17.8, 80.5)
- added REF**: VIA-0.6mm, Logan:VIA-0.6mm, F.Cu at (21.8, 79.5)
- added REF**: VIA-0.6mm, Logan:VIA-0.6mm, F.Cu at (20.8, 79.5)
- added REF**: VIA-0.6mm, Logan:VIA-0.6mm, F.Cu at (19.8, 79.5)
- added REF**: VIA-0.6mm, Logan:VIA-0.6mm, F.Cu at (18.8, 79.5)
- added REF**: VIA-0.6mm, Logan:VIA-0.6mm, F.Cu at (17.8, 79.5)
- added REF**: VIA-0.6mm, Logan:VIA-0.6mm, F.Cu at (65.0, 77.0)
- added REF**: VIA-0.6mm, Logan:VIA-0.6mm, F.Cu at (64.0, 77.0)
- added REF**: VIA-0.6mm, Logan:VIA-0.6mm, F.Cu at (63.0, 77.0)
- added REF**: VIA-0.6mm, Logan:VIA-0.6mm, F.Cu at (62.0, 77.0)
- added REF**: VIA-0.6mm, Logan:VIA-0.6mm, F.Cu at (19.8, 83.5)
- added REF**: VIA-0.6mm, Logan:VIA-0.6mm, F.Cu at (61.0, 77.0)
- added REF**: VIA-0.6mm, Logan:VIA-0.6mm, F.Cu at (60.0, 77.0)
- added REF**: VIA-0.6mm, Logan:VIA-0.6mm, F.Cu at (59.0, 77.0)
- added REF**: VIA-0.6mm, Logan:VIA-0.6mm, F.Cu at (58.0, 77.0)
- added REF**: VIA-0.6mm, Logan:VIA-0.6mm, F.Cu at (57.0, 77.0)
- added REF**: VIA-0.6mm, Logan:VIA-0.6mm, F.Cu at (65.0, 76.0)
- added REF**: VIA-0.6mm, Logan:VIA-0.6mm, F.Cu at (64.0, 76.0)
- added REF**: VIA-0.6mm, Logan:VIA-0.6mm, F.Cu at (63.0, 76.0)
- added REF**: VIA-0.6mm, Logan:VIA-0.6mm, F.Cu at (62.0, 76.0)
- added REF**: VIA-0.6mm, Logan:VIA-0.6mm, F.Cu at (61.0, 76.0)
- added REF**: VIA-0.6mm, Logan:VIA-0.6mm, F.Cu at (18.8, 83.5)
- added REF**: VIA-0.6mm, Logan:VIA-0.6mm, F.Cu at (60.0, 76.0)
- added REF**: VIA-0.6mm, Logan:VIA-0.6mm, F.Cu at (59.0, 76.0)
- added REF**: VIA-0.6mm, Logan:VIA-0.6mm, F.Cu at (58.0, 76.0)
- added REF**: VIA-0.6mm, Logan:VIA-0.6mm, F.Cu at (57.0, 76.0)
- added REF**: VIA-0.6mm, Logan:VIA-0.6mm, F.Cu at (21.8, 71.0)
- added REF**: VIA-0.6mm, Logan:VIA-0.6mm, F.Cu at (20.8, 71.0)
- added REF**: VIA-0.6mm, Logan:VIA-0.6mm, F.Cu at (19.8, 71.0)
- added REF**: VIA-0.6mm, Logan:VIA-0.6mm, F.Cu at (18.8, 71.0)
- added REF**: VIA-0.6mm, Logan:VIA-0.6mm, F.Cu at (17.8, 71.0)
- added REF**: VIA-0.6mm, Logan:VIA-0.6mm, F.Cu at (65.0, 75.0)
- added REF**: VIA-0.6mm, Logan:VIA-0.6mm, F.Cu at (17.8, 83.5)
- added REF**: VIA-0.6mm, Logan:VIA-0.6mm, F.Cu at (64.0, 75.0)
- added REF**: VIA-0.6mm, Logan:VIA-0.6mm, F.Cu at (63.0, 75.0)
- added REF**: VIA-0.6mm, Logan:VIA-0.6mm, F.Cu at (62.0, 75.0)
- added REF**: VIA-0.6mm, Logan:VIA-0.6mm, F.Cu at (61.0, 75.0)
- added REF**: VIA-0.6mm, Logan:VIA-0.6mm, F.Cu at (60.0, 75.0)
- added REF**: VIA-0.6mm, Logan:VIA-0.6mm, F.Cu at (59.0, 75.0)
- added REF**: VIA-0.6mm, Logan:VIA-0.6mm, F.Cu at (58.0, 75.0)
- added REF**: VIA-0.6mm, Logan:VIA-0.6mm, F.Cu at (57.0, 75.0)
- added REF**: VIA-0.6mm, Logan:VIA-0.6mm, F.Cu at (21.8, 70.0)
- added REF**: VIA-0.6mm, Logan:VIA-0.6mm, F.Cu at (20.8, 70.0)
- added REF**: VIA-0.6mm, Logan:VIA-0.6mm, F.Cu at (21.8, 82.5)
- added REF**: VIA-0.6mm, Logan:VIA-0.6mm, F.Cu at (19.8, 70.0)
- added REF**: VIA-0.6mm, Logan:VIA-0.6mm, F.Cu at (18.8, 70.0)
- added REF**: VIA-0.6mm, Logan:VIA-0.6mm, F.Cu at (17.8, 70.0)
- added REF**: VIA-0.6mm, Logan:VIA-0.6mm, F.Cu at (65.0, 74.0)
- added REF**: VIA-0.6mm, Logan:VIA-0.6mm, F.Cu at (64.0, 74.0)
- added REF**: VIA-0.6mm, Logan:VIA-0.6mm, F.Cu at (63.0, 74.0)
- added REF**: VIA-0.6mm, Logan:VIA-0.6mm, F.Cu at (59.0, 74.0)
- added REF**: VIA-0.6mm, Logan:VIA-0.6mm, F.Cu at (58.0, 74.0)
- added REF**: VIA-0.6mm, Logan:VIA-0.6mm, F.Cu at (57.0, 74.0)
- added REF**: VIA-0.6mm, Logan:VIA-0.6mm, F.Cu at (21.8, 69.0)
- added REF**: VIA-0.6mm, Logan:VIA-0.6mm, F.Cu at (20.8, 82.5)
- added REF**: VIA-0.6mm, Logan:VIA-0.6mm, F.Cu at (20.8, 69.0)
- added REF**: VIA-0.6mm, Logan:VIA-0.6mm, F.Cu at (19.8, 69.0)
- added REF**: VIA-0.6mm, Logan:VIA-0.6mm, F.Cu at (18.8, 69.0)
- added REF**: VIA-0.6mm, Logan:VIA-0.6mm, F.Cu at (17.8, 69.0)
- added REF**: VIA-0.6mm, Logan:VIA-0.6mm, F.Cu at (65.0, 73.0)
- added REF**: VIA-0.6mm, Logan:VIA-0.6mm, F.Cu at (64.0, 73.0)
- added REF**: VIA-0.6mm, Logan:VIA-0.6mm, F.Cu at (63.0, 73.0)
- added REF**: VIA-0.6mm, Logan:VIA-0.6mm, F.Cu at (59.0, 73.0)
- added REF**: VIA-0.6mm, Logan:VIA-0.6mm, F.Cu at (58.0, 73.0)
- added REF**: VIA-0.6mm, Logan:VIA-0.6mm, F.Cu at (57.0, 73.0)
- added REF**: VIA-0.6mm, Logan:VIA-0.6mm, F.Cu at (19.8, 82.5)
- added REF**: VIA-0.6mm, Logan:VIA-0.6mm, F.Cu at (21.8, 68.0)
- added REF**: VIA-0.6mm, Logan:VIA-0.6mm, F.Cu at (20.8, 68.0)
- added REF**: VIA-0.6mm, Logan:VIA-0.6mm, F.Cu at (19.8, 68.0)
- added REF**: VIA-0.6mm, Logan:VIA-0.6mm, F.Cu at (18.8, 68.0)
- added REF**: VIA-0.6mm, Logan:VIA-0.6mm, F.Cu at (17.8, 68.0)
- added REF**: VIA-0.6mm, Logan:VIA-0.6mm, F.Cu at (65.0, 72.0)
- added REF**: VIA-0.6mm, Logan:VIA-0.6mm, F.Cu at (64.0, 72.0)
- added REF**: VIA-0.6mm, Logan:VIA-0.6mm, F.Cu at (63.0, 72.0)
- added REF**: VIA-0.6mm, Logan:VIA-0.6mm, F.Cu at (59.0, 72.0)
- added REF**: VIA-0.6mm, Logan:VIA-0.6mm, F.Cu at (58.0, 72.0)
- added REF**: VIA-0.6mm, Logan:VIA-0.6mm, F.Cu at (18.8, 82.5)
- added REF**: VIA-0.6mm, Logan:VIA-0.6mm, F.Cu at (57.0, 72.0)
- Q2: value MMBT3904 -> BUK9515-60E; footprint Package_TO_SOT_SMD:SOT-23 -> Package_TO_SOT_THT:TO-220-3_Vertical
- TP1, TP2, TP3: footprint TestPoint:TestPoint_Pad_D2.0mm -> TestPoint:TestPoint_THTPad_D1.5mm_Drill0.7mm
- moved RV1 103.8 mm to (49.9, 93.2)
- moved Q2 48.0 mm to (82.8, 74.9), turned to 270 degrees
- moved R11 40.7 mm to (49.6, 96.6), turned to 180 degrees
- moved TP8 32.9 mm to (50.6, 81.1)
- moved TP5 30.8 mm to (52.8, 75.7)
- moved C2 29.8 mm to (73.6, 72.4), turned to 270 degrees
- moved TP4 29.7 mm to (50.1, 74.3)
- moved TP7 29.6 mm to (47.6, 81.3)
- moved DS1 26.5 mm to (19.4, 102.2)
- moved U7 26.5 mm to (36.5, 95.0)
- moved TP12 23.7 mm to (75.2, 84.6)
- moved TP13 20.7 mm to (79.1, 86.2)
- moved TP11 20.4 mm to (66.0, 78.8)
- moved TP9 15.2 mm to (51.7, 84.9)
- moved J3 14.6 mm to (106.1, 96.4)
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Connections:
- J1 pad 9: Net-(J1-Pad9) -> GND
- Q2 pad 1: Net-(Q2-Pad1) -> Net-(Q1-Pad1)
- Q2 pad 2: Net-(Q2-Pad2) -> /DC Driver/OUT+
- Q2 pad 3: Net-(DS1-Pad16) -> Net-(Q1-Pad2)
- U2 pad 1: Net-(U2-Pad1) -> /LCD/EN
- U2 pad 2: Net-(U2-Pad2) -> /LCD/Data
- U2 pad 29: /LCD/Data -> Net-(U2-Pad29)
- U2 pad 3: Net-(U2-Pad3) -> /LCD/CLK
- U2 pad 30: /LCD/CLK -> Net-(U2-Pad30)
- U2 pad 31: /LCD/EN -> Net-(U2-Pad31)
Routing:
- net Net-(DS1-Pad3): track 0.00 -> 46.4 mm
- net Net-(Q1-Pad1): track 0.00 -> 29.5 mm
- net /LCD/EN: track 0.00 -> 26.1 mm
- net NEUT: track 0.00 -> 23.9 mm
- net /Microcontroller/ADC_in0: track 0.00 -> 22.6 mm
- net /Microcontroller/~RESET: track 0.00 -> 22.6 mm
- net /Microcontroller/SWDIO: track 0.00 -> 22.3 mm
- net /LCD/D7: track 0.00 -> 20.0 mm
- net /DC Driver/~CS: track 0.00 -> 19.7 mm, vias 0 -> 2
- net /LCD/D6: track 0.00 -> 18.7 mm
- net /LCD/D5: track 0.00 -> 17.5 mm
- net /LCD/CLK: track 0.00 -> 17.3 mm
- net /DC Driver/SCK: track 0.00 -> 16.6 mm, vias 0 -> 2
- net /LCD/D4: track 0.00 -> 16.5 mm, vias 0 -> 1
- net /Microcontroller/SWCLK: track 0.00 -> 16.0 mm
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- added copper zone on 5V0, net +5V
- added copper zone on F.Cu, net +5V
- added copper zone on F.Cu, net /DC Driver/OUT+
- added copper zone on B.Cu, net 3V3
- added copper zone on F.Cu, net 3V3
- added copper zone on F.Cu, net GND
- added copper zone on GND, net GND
- added copper zone on F.Cu, net Net-(Q1-Pad2)
Other:
- board outline added: 101 x 64 mm
- copper layers 2 -> 4

Commit message: Laptop
Parts:
- added C14: 0.01u, Capacitor_SMD:C_0603_1608Metric, F.Cu at (32.8, 77.0)
- added C8: 0.01u, Capacitor_SMD:C_0603_1608Metric, F.Cu at (32.8, 74.0)
- added R12: 10k, Resistor_SMD:R_0603_1608Metric, F.Cu at (23.0, 98.2)
- added R13: 10k, Resistor_SMD:R_0603_1608Metric, F.Cu at (23.0, 93.0)
- added R14: 10k, Resistor_SMD:R_0603_1608Metric, F.Cu at (32.8, 75.5)
- added R15: 10k, Resistor_SMD:R_0603_1608Metric, F.Cu at (32.8, 78.5)
- added R16: 10k, Resistor_SMD:R_0603_1608Metric, F.Cu at (23.0, 90.5)
- added REF**: VIA-0.6mm, Logan:VIA-0.6mm, F.Cu at (115.2, 103.8)
- added REF**: VIA-0.6mm, Logan:VIA-0.6mm, F.Cu at (106.2, 103.8)
- added REF**: VIA-0.6mm, Logan:VIA-0.6mm, F.Cu at (82.2, 101.8)
- added REF**: VIA-0.6mm, Logan:VIA-0.6mm, F.Cu at (81.2, 101.8)
- added REF**: VIA-0.6mm, Logan:VIA-0.6mm, F.Cu at (80.2, 101.8)
- added REF**: VIA-0.6mm, Logan:VIA-0.6mm, F.Cu at (79.2, 101.8)
- added REF**: VIA-0.6mm, Logan:VIA-0.6mm, F.Cu at (78.2, 101.8)
- added REF**: VIA-0.6mm, Logan:VIA-0.6mm, F.Cu at (77.2, 101.8)
- added REF**: VIA-0.6mm, Logan:VIA-0.6mm, F.Cu at (76.2, 101.8)
- added REF**: VIA-0.6mm, Logan:VIA-0.6mm, F.Cu at (115.2, 100.8)
- added REF**: VIA-0.6mm, Logan:VIA-0.6mm, F.Cu at (114.2, 100.8)
- added REF**: VIA-0.6mm, Logan:VIA-0.6mm, F.Cu at (113.2, 100.8)
- added REF**: VIA-0.6mm, Logan:VIA-0.6mm, F.Cu at (105.2, 103.8)
- added REF**: VIA-0.6mm, Logan:VIA-0.6mm, F.Cu at (112.2, 100.8)
- added REF**: VIA-0.6mm, Logan:VIA-0.6mm, F.Cu at (111.2, 100.8)
- added REF**: VIA-0.6mm, Logan:VIA-0.6mm, F.Cu at (110.2, 100.8)
- added REF**: VIA-0.6mm, Logan:VIA-0.6mm, F.Cu at (102.2, 100.8)
- added REF**: VIA-0.6mm, Logan:VIA-0.6mm, F.Cu at (101.2, 100.8)
- added REF**: VIA-0.6mm, Logan:VIA-0.6mm, F.Cu at (100.2, 100.8)
- added REF**: VIA-0.6mm, Logan:VIA-0.6mm, F.Cu at (99.2, 100.8)
- added REF**: VIA-0.6mm, Logan:VIA-0.6mm, F.Cu at (98.2, 100.8)
- added REF**: VIA-0.6mm, Logan:VIA-0.6mm, F.Cu at (97.2, 100.8)
- added REF**: VIA-0.6mm, Logan:VIA-0.6mm, F.Cu at (96.2, 100.8)
- added REF**: VIA-0.6mm, Logan:VIA-0.6mm, F.Cu at (104.2, 103.8)
- added REF**: VIA-0.6mm, Logan:VIA-0.6mm, F.Cu at (95.2, 100.8)
- added REF**: VIA-0.6mm, Logan:VIA-0.6mm, F.Cu at (94.2, 100.8)
- added REF**: VIA-0.6mm, Logan:VIA-0.6mm, F.Cu at (93.2, 100.8)
- added REF**: VIA-0.6mm, Logan:VIA-0.6mm, F.Cu at (92.2, 100.8)
- added REF**: VIA-0.6mm, Logan:VIA-0.6mm, F.Cu at (91.2, 100.8)
- added REF**: VIA-0.6mm, Logan:VIA-0.6mm, F.Cu at (90.2, 100.8)
- added REF**: VIA-0.6mm, Logan:VIA-0.6mm, F.Cu at (89.2, 100.8)
- added REF**: VIA-0.6mm, Logan:VIA-0.6mm, F.Cu at (88.2, 100.8)
- added REF**: VIA-0.6mm, Logan:VIA-0.6mm, F.Cu at (87.2, 100.8)
- added REF**: VIA-0.6mm, Logan:VIA-0.6mm, F.Cu at (86.2, 100.8)
- added REF**: VIA-0.6mm, Logan:VIA-0.6mm, F.Cu at (103.2, 103.8)
- added REF**: VIA-0.6mm, Logan:VIA-0.6mm, F.Cu at (85.2, 100.8)
- added REF**: VIA-0.6mm, Logan:VIA-0.6mm, F.Cu at (84.2, 100.8)
- added REF**: VIA-0.6mm, Logan:VIA-0.6mm, F.Cu at (83.2, 100.8)
- added REF**: VIA-0.6mm, Logan:VIA-0.6mm, F.Cu at (82.2, 100.8)
- added REF**: VIA-0.6mm, Logan:VIA-0.6mm, F.Cu at (81.2, 100.8)
- added REF**: VIA-0.6mm, Logan:VIA-0.6mm, F.Cu at (80.2, 100.8)
- added REF**: VIA-0.6mm, Logan:VIA-0.6mm, F.Cu at (79.2, 100.8)
- added REF**: VIA-0.6mm, Logan:VIA-0.6mm, F.Cu at (78.2, 100.8)
- added REF**: VIA-0.6mm, Logan:VIA-0.6mm, F.Cu at (77.2, 100.8)
- added REF**: VIA-0.6mm, Logan:VIA-0.6mm, F.Cu at (76.2, 100.8)
- added REF**: VIA-0.6mm, Logan:VIA-0.6mm, F.Cu at (102.2, 103.8)
- added REF**: VIA-0.6mm, Logan:VIA-0.6mm, F.Cu at (115.2, 99.8)
- added REF**: VIA-0.6mm, Logan:VIA-0.6mm, F.Cu at (114.2, 99.8)
- added REF**: VIA-0.6mm, Logan:VIA-0.6mm, F.Cu at (113.2, 99.8)
- added REF**: VIA-0.6mm, Logan:VIA-0.6mm, F.Cu at (112.2, 99.8)
- added REF**: VIA-0.6mm, Logan:VIA-0.6mm, F.Cu at (111.2, 99.8)
- added REF**: VIA-0.6mm, Logan:VIA-0.6mm, F.Cu at (110.2, 99.8)
- added REF**: VIA-0.6mm, Logan:VIA-0.6mm, F.Cu at (102.2, 99.8)
- added REF**: VIA-0.6mm, Logan:VIA-0.6mm, F.Cu at (101.2, 99.8)
- added REF**: VIA-0.6mm, Logan:VIA-0.6mm, F.Cu at (100.2, 99.8)
- added REF**: VIA-0.6mm, Logan:VIA-0.6mm, F.Cu at (99.2, 99.8)
- added REF**: VIA-0.6mm, Logan:VIA-0.6mm, F.Cu at (101.2, 103.8)
- added REF**: VIA-0.6mm, Logan:VIA-0.6mm, F.Cu at (98.2, 99.8)
- added REF**: VIA-0.6mm, Logan:VIA-0.6mm, F.Cu at (97.2, 99.8)
- added REF**: VIA-0.6mm, Logan:VIA-0.6mm, F.Cu at (96.2, 99.8)
- added REF**: VIA-0.6mm, Logan:VIA-0.6mm, F.Cu at (95.2, 99.8)
- added REF**: VIA-0.6mm, Logan:VIA-0.6mm, F.Cu at (94.2, 99.8)
- added REF**: VIA-0.6mm, Logan:VIA-0.6mm, F.Cu at (93.2, 99.8)
- added REF**: VIA-0.6mm, Logan:VIA-0.6mm, F.Cu at (92.2, 99.8)
- added REF**: VIA-0.6mm, Logan:VIA-0.6mm, F.Cu at (91.2, 99.8)
- added REF**: VIA-0.6mm, Logan:VIA-0.6mm, F.Cu at (90.2, 99.8)
- added REF**: VIA-0.6mm, Logan:VIA-0.6mm, F.Cu at (89.2, 99.8)
- added REF**: VIA-0.6mm, Logan:VIA-0.6mm, F.Cu at (100.2, 103.8)
- added REF**: VIA-0.6mm, Logan:VIA-0.6mm, F.Cu at (88.2, 99.8)
- added REF**: VIA-0.6mm, Logan:VIA-0.6mm, F.Cu at (87.2, 99.8)
- added REF**: VIA-0.6mm, Logan:VIA-0.6mm, F.Cu at (86.2, 99.8)
- added REF**: VIA-0.6mm, Logan:VIA-0.6mm, F.Cu at (85.2, 99.8)
- added REF**: VIA-0.6mm, Logan:VIA-0.6mm, F.Cu at (84.2, 99.8)
- added REF**: VIA-0.6mm, Logan:VIA-0.6mm, F.Cu at (83.2, 99.8)
- added REF**: VIA-0.6mm, Logan:VIA-0.6mm, F.Cu at (82.2, 99.8)
- added REF**: VIA-0.6mm, Logan:VIA-0.6mm, F.Cu at (81.2, 99.8)
- added REF**: VIA-0.6mm, Logan:VIA-0.6mm, F.Cu at (80.2, 99.8)
- added REF**: VIA-0.6mm, Logan:VIA-0.6mm, F.Cu at (79.2, 99.8)
- added REF**: VIA-0.6mm, Logan:VIA-0.6mm, F.Cu at (99.2, 103.8)
- added REF**: VIA-0.6mm, Logan:VIA-0.6mm, F.Cu at (78.2, 99.8)
- added REF**: VIA-0.6mm, Logan:VIA-0.6mm, F.Cu at (77.2, 99.8)
- added REF**: VIA-0.6mm, Logan:VIA-0.6mm, F.Cu at (76.2, 99.8)
- added REF**: VIA-0.6mm, Logan:VIA-0.6mm, F.Cu at (115.2, 98.8)
- added REF**: VIA-0.6mm, Logan:VIA-0.6mm, F.Cu at (114.2, 98.8)
- added REF**: VIA-0.6mm, Logan:VIA-0.6mm, F.Cu at (113.2, 98.8)
- added REF**: VIA-0.6mm, Logan:VIA-0.6mm, F.Cu at (112.2, 98.8)
- added REF**: VIA-0.6mm, Logan:VIA-0.6mm, F.Cu at (111.2, 98.8)
- added REF**: VIA-0.6mm, Logan:VIA-0.6mm, F.Cu at (110.2, 98.8)
- added REF**: VIA-0.6mm, Logan:VIA-0.6mm, F.Cu at (102.2, 98.8)
- added REF**: VIA-0.6mm, Logan:VIA-0.6mm, F.Cu at (98.2, 103.8)
- added REF**: VIA-0.6mm, Logan:VIA-0.6mm, F.Cu at (101.2, 98.8)
- added REF**: VIA-0.6mm, Logan:VIA-0.6mm, F.Cu at (100.2, 98.8)
- added REF**: VIA-0.6mm, Logan:VIA-0.6mm, F.Cu at (99.2, 98.8)
- added REF**: VIA-0.6mm, Logan:VIA-0.6mm, F.Cu at (98.2, 98.8)
- added REF**: VIA-0.6mm, Logan:VIA-0.6mm, F.Cu at (97.2, 98.8)
- added REF**: VIA-0.6mm, Logan:VIA-0.6mm, F.Cu at (96.2, 98.8)
- added REF**: VIA-0.6mm, Logan:VIA-0.6mm, F.Cu at (95.2, 98.8)
- added REF**: VIA-0.6mm, Logan:VIA-0.6mm, F.Cu at (94.2, 98.8)
- added REF**: VIA-0.6mm, Logan:VIA-0.6mm, F.Cu at (93.2, 98.8)
- added REF**: VIA-0.6mm, Logan:VIA-0.6mm, F.Cu at (92.2, 98.8)
- added REF**: VIA-0.6mm, Logan:VIA-0.6mm, F.Cu at (97.2, 103.8)
- added REF**: VIA-0.6mm, Logan:VIA-0.6mm, F.Cu at (91.2, 98.8)
- added REF**: VIA-0.6mm, Logan:VIA-0.6mm, F.Cu at (90.2, 98.8)
- added REF**: VIA-0.6mm, Logan:VIA-0.6mm, F.Cu at (89.2, 98.8)
- added REF**: VIA-0.6mm, Logan:VIA-0.6mm, F.Cu at (88.2, 98.8)
- added REF**: VIA-0.6mm, Logan:VIA-0.6mm, F.Cu at (87.2, 98.8)
- added REF**: VIA-0.6mm, Logan:VIA-0.6mm, F.Cu at (86.2, 98.8)
- added REF**: VIA-0.6mm, Logan:VIA-0.6mm, F.Cu at (85.2, 98.8)
- added REF**: VIA-0.6mm, Logan:VIA-0.6mm, F.Cu at (84.2, 98.8)
- added REF**: VIA-0.6mm, Logan:VIA-0.6mm, F.Cu at (83.2, 98.8)
- added REF**: VIA-0.6mm, Logan:VIA-0.6mm, F.Cu at (82.2, 98.8)
- added REF**: VIA-0.6mm, Logan:VIA-0.6mm, F.Cu at (114.2, 103.8)
- added REF**: VIA-0.6mm, Logan:VIA-0.6mm, F.Cu at (96.2, 103.8)
- added REF**: VIA-0.6mm, Logan:VIA-0.6mm, F.Cu at (81.2, 98.8)
- added REF**: VIA-0.6mm, Logan:VIA-0.6mm, F.Cu at (80.2, 98.8)
- added REF**: VIA-0.6mm, Logan:VIA-0.6mm, F.Cu at (79.2, 98.8)
- added REF**: VIA-0.6mm, Logan:VIA-0.6mm, F.Cu at (78.2, 98.8)
- added REF**: VIA-0.6mm, Logan:VIA-0.6mm, F.Cu at (77.2, 98.8)
- added REF**: VIA-0.6mm, Logan:VIA-0.6mm, F.Cu at (76.2, 98.8)
- added REF**: VIA-0.6mm, Logan:VIA-0.6mm, F.Cu at (115.2, 97.8)
- added REF**: VIA-0.6mm, Logan:VIA-0.6mm, F.Cu at (114.2, 97.8)
- added REF**: VIA-0.6mm, Logan:VIA-0.6mm, F.Cu at (113.2, 97.8)
- added REF**: VIA-0.6mm, Logan:VIA-0.6mm, F.Cu at (112.2, 97.8)
- added REF**: VIA-0.6mm, Logan:VIA-0.6mm, F.Cu at (95.2, 103.8)
- added REF**: VIA-0.6mm, Logan:VIA-0.6mm, F.Cu at (111.2, 97.8)
- added REF**: VIA-0.6mm, Logan:VIA-0.6mm, F.Cu at (110.2, 97.8)
- added REF**: VIA-0.6mm, Logan:VIA-0.6mm, F.Cu at (102.2, 97.8)
- added REF**: VIA-0.6mm, Logan:VIA-0.6mm, F.Cu at (101.2, 97.8)
- added REF**: VIA-0.6mm, Logan:VIA-0.6mm, F.Cu at (100.2, 97.8)
- added REF**: VIA-0.6mm, Logan:VIA-0.6mm, F.Cu at (99.2, 97.8)
- added REF**: VIA-0.6mm, Logan:VIA-0.6mm, F.Cu at (98.2, 97.8)
- added REF**: VIA-0.6mm, Logan:VIA-0.6mm, F.Cu at (97.2, 97.8)
- added REF**: VIA-0.6mm, Logan:VIA-0.6mm, F.Cu at (96.2, 97.8)
- added REF**: VIA-0.6mm, Logan:VIA-0.6mm, F.Cu at (95.2, 97.8)
- added REF**: VIA-0.6mm, Logan:VIA-0.6mm, F.Cu at (94.2, 103.8)
- added REF**: VIA-0.6mm, Logan:VIA-0.6mm, F.Cu at (94.2, 97.8)
- added REF**: VIA-0.6mm, Logan:VIA-0.6mm, F.Cu at (93.2, 97.8)
- added REF**: VIA-0.6mm, Logan:VIA-0.6mm, F.Cu at (92.2, 97.8)
- added REF**: VIA-0.6mm, Logan:VIA-0.6mm, F.Cu at (91.2, 97.8)
- added REF**: VIA-0.6mm, Logan:VIA-0.6mm, F.Cu at (90.2, 97.8)
- added REF**: VIA-0.6mm, Logan:VIA-0.6mm, F.Cu at (89.2, 97.8)
- added REF**: VIA-0.6mm, Logan:VIA-0.6mm, F.Cu at (88.2, 97.8)
- added REF**: VIA-0.6mm, Logan:VIA-0.6mm, F.Cu at (87.2, 97.8)
- added REF**: VIA-0.6mm, Logan:VIA-0.6mm, F.Cu at (86.2, 97.8)
- added REF**: VIA-0.6mm, Logan:VIA-0.6mm, F.Cu at (85.2, 97.8)
- added REF**: VIA-0.6mm, Logan:VIA-0.6mm, F.Cu at (93.2, 103.8)
- added REF**: VIA-0.6mm, Logan:VIA-0.6mm, F.Cu at (84.2, 97.8)
- added REF**: VIA-0.6mm, Logan:VIA-0.6mm, F.Cu at (83.2, 97.8)
- added REF**: VIA-0.6mm, Logan:VIA-0.6mm, F.Cu at (82.2, 97.8)
- added REF**: VIA-0.6mm, Logan:VIA-0.6mm, F.Cu at (81.2, 97.8)
- added REF**: VIA-0.6mm, Logan:VIA-0.6mm, F.Cu at (80.2, 97.8)
- added REF**: VIA-0.6mm, Logan:VIA-0.6mm, F.Cu at (79.2, 97.8)
- added REF**: VIA-0.6mm, Logan:VIA-0.6mm, F.Cu at (78.2, 97.8)
- added REF**: VIA-0.6mm, Logan:VIA-0.6mm, F.Cu at (77.2, 97.8)
- added REF**: VIA-0.6mm, Logan:VIA-0.6mm, F.Cu at (76.2, 97.8)
- added REF**: VIA-0.6mm, Logan:VIA-0.6mm, F.Cu at (115.2, 96.8)
- added REF**: VIA-0.6mm, Logan:VIA-0.6mm, F.Cu at (92.2, 103.8)
- added REF**: VIA-0.6mm, Logan:VIA-0.6mm, F.Cu at (114.2, 96.8)
- added REF**: VIA-0.6mm, Logan:VIA-0.6mm, F.Cu at (100.2, 96.8)
- added REF**: VIA-0.6mm, Logan:VIA-0.6mm, F.Cu at (99.2, 96.8)
- added REF**: VIA-0.6mm, Logan:VIA-0.6mm, F.Cu at (98.2, 96.8)
- added REF**: VIA-0.6mm, Logan:VIA-0.6mm, F.Cu at (97.2, 96.8)
- added REF**: VIA-0.6mm, Logan:VIA-0.6mm, F.Cu at (96.2, 96.8)
- added REF**: VIA-0.6mm, Logan:VIA-0.6mm, F.Cu at (95.2, 96.8)
- added REF**: VIA-0.6mm, Logan:VIA-0.6mm, F.Cu at (94.2, 96.8)
- added REF**: VIA-0.6mm, Logan:VIA-0.6mm, F.Cu at (93.2, 96.8)
- added REF**: VIA-0.6mm, Logan:VIA-0.6mm, F.Cu at (92.2, 96.8)
- added REF**: VIA-0.6mm, Logan:VIA-0.6mm, F.Cu at (91.2, 103.8)
- added REF**: VIA-0.6mm, Logan:VIA-0.6mm, F.Cu at (91.2, 96.8)
- added REF**: VIA-0.6mm, Logan:VIA-0.6mm, F.Cu at (90.2, 96.8)
- added REF**: VIA-0.6mm, Logan:VIA-0.6mm, F.Cu at (89.2, 96.8)
- added REF**: VIA-0.6mm, Logan:VIA-0.6mm, F.Cu at (88.2, 96.8)
- added REF**: VIA-0.6mm, Logan:VIA-0.6mm, F.Cu at (87.2, 96.8)
- added REF**: VIA-0.6mm, Logan:VIA-0.6mm, F.Cu at (86.2, 96.8)
- added REF**: VIA-0.6mm, Logan:VIA-0.6mm, F.Cu at (85.2, 96.8)
- added REF**: VIA-0.6mm, Logan:VIA-0.6mm, F.Cu at (84.2, 96.8)
- added REF**: VIA-0.6mm, Logan:VIA-0.6mm, F.Cu at (83.2, 96.8)
- added REF**: VIA-0.6mm, Logan:VIA-0.6mm, F.Cu at (82.2, 96.8)
- added REF**: VIA-0.6mm, Logan:VIA-0.6mm, F.Cu at (90.2, 103.8)
- added REF**: VIA-0.6mm, Logan:VIA-0.6mm, F.Cu at (81.2, 96.8)
- added REF**: VIA-0.6mm, Logan:VIA-0.6mm, F.Cu at (80.2, 96.8)
- added REF**: VIA-0.6mm, Logan:VIA-0.6mm, F.Cu at (79.2, 96.8)
- added REF**: VIA-0.6mm, Logan:VIA-0.6mm, F.Cu at (78.2, 96.8)
- added REF**: VIA-0.6mm, Logan:VIA-0.6mm, F.Cu at (77.2, 96.8)
- added REF**: VIA-0.6mm, Logan:VIA-0.6mm, F.Cu at (76.2, 96.8)
- added REF**: VIA-0.6mm, Logan:VIA-0.6mm, F.Cu at (115.2, 95.8)
- added REF**: VIA-0.6mm, Logan:VIA-0.6mm, F.Cu at (114.2, 95.8)
- added REF**: VIA-0.6mm, Logan:VIA-0.6mm, F.Cu at (100.2, 95.8)
- added REF**: VIA-0.6mm, Logan:VIA-0.6mm, F.Cu at (99.2, 95.8)
- added REF**: VIA-0.6mm, Logan:VIA-0.6mm, F.Cu at (89.2, 103.8)
- added REF**: VIA-0.6mm, Logan:VIA-0.6mm, F.Cu at (98.2, 95.8)
- added REF**: VIA-0.6mm, Logan:VIA-0.6mm, F.Cu at (97.2, 95.8)
- added REF**: VIA-0.6mm, Logan:VIA-0.6mm, F.Cu at (96.2, 95.8)
- added REF**: VIA-0.6mm, Logan:VIA-0.6mm, F.Cu at (95.2, 95.8)
- added REF**: VIA-0.6mm, Logan:VIA-0.6mm, F.Cu at (94.2, 95.8)
- added REF**: VIA-0.6mm, Logan:VIA-0.6mm, F.Cu at (93.2, 95.8)
- added REF**: VIA-0.6mm, Logan:VIA-0.6mm, F.Cu at (92.2, 95.8)
- added REF**: VIA-0.6mm, Logan:VIA-0.6mm, F.Cu at (91.2, 95.8)
- added REF**: VIA-0.6mm, Logan:VIA-0.6mm, F.Cu at (90.2, 95.8)
- added REF**: VIA-0.6mm, Logan:VIA-0.6mm, F.Cu at (89.2, 95.8)
- added REF**: VIA-0.6mm, Logan:VIA-0.6mm, F.Cu at (88.2, 103.8)
- added REF**: VIA-0.6mm, Logan:VIA-0.6mm, F.Cu at (88.2, 95.8)
- added REF**: VIA-0.6mm, Logan:VIA-0.6mm, F.Cu at (87.2, 95.8)
- added REF**: VIA-0.6mm, Logan:VIA-0.6mm, F.Cu at (86.2, 95.8)
- added REF**: VIA-0.6mm, Logan:VIA-0.6mm, F.Cu at (85.2, 95.8)
- added REF**: VIA-0.6mm, Logan:VIA-0.6mm, F.Cu at (84.2, 95.8)
- added REF**: VIA-0.6mm, Logan:VIA-0.6mm, F.Cu at (83.2, 95.8)
- added REF**: VIA-0.6mm, Logan:VIA-0.6mm, F.Cu at (82.2, 95.8)
- added REF**: VIA-0.6mm, Logan:VIA-0.6mm, F.Cu at (81.2, 95.8)
- added REF**: VIA-0.6mm, Logan:VIA-0.6mm, F.Cu at (80.2, 95.8)
- added REF**: VIA-0.6mm, Logan:VIA-0.6mm, F.Cu at (79.2, 95.8)
- added REF**: VIA-0.6mm, Logan:VIA-0.6mm, F.Cu at (87.2, 103.8)
- added REF**: VIA-0.6mm, Logan:VIA-0.6mm, F.Cu at (78.2, 95.8)
- added REF**: VIA-0.6mm, Logan:VIA-0.6mm, F.Cu at (77.2, 95.8)
- added REF**: VIA-0.6mm, Logan:VIA-0.6mm, F.Cu at (76.2, 95.8)
- added REF**: VIA-0.6mm, Logan:VIA-0.6mm, F.Cu at (115.2, 94.8)
- added REF**: VIA-0.6mm, Logan:VIA-0.6mm, F.Cu at (114.2, 94.8)
- added REF**: VIA-0.6mm, Logan:VIA-0.6mm, F.Cu at (100.2, 94.8)
- added REF**: VIA-0.6mm, Logan:VIA-0.6mm, F.Cu at (99.2, 94.8)
- added REF**: VIA-0.6mm, Logan:VIA-0.6mm, F.Cu at (98.2, 94.8)
- added REF**: VIA-0.6mm, Logan:VIA-0.6mm, F.Cu at (97.2, 94.8)
- added REF**: VIA-0.6mm, Logan:VIA-0.6mm, F.Cu at (96.2, 94.8)
- added REF**: VIA-0.6mm, Logan:VIA-0.6mm, F.Cu at (113.2, 103.8)
- added REF**: VIA-0.6mm, Logan:VIA-0.6mm, F.Cu at (86.2, 103.8)
- added REF**: VIA-0.6mm, Logan:VIA-0.6mm, F.Cu at (95.2, 94.8)
- added REF**: VIA-0.6mm, Logan:VIA-0.6mm, F.Cu at (94.2, 94.8)
- added REF**: VIA-0.6mm, Logan:VIA-0.6mm, F.Cu at (93.2, 94.8)
- added REF**: VIA-0.6mm, Logan:VIA-0.6mm, F.Cu at (92.2, 94.8)
- added REF**: VIA-0.6mm, Logan:VIA-0.6mm, F.Cu at (91.2, 94.8)
- added REF**: VIA-0.6mm, Logan:VIA-0.6mm, F.Cu at (90.2, 94.8)
- added REF**: VIA-0.6mm, Logan:VIA-0.6mm, F.Cu at (89.2, 94.8)
- added REF**: VIA-0.6mm, Logan:VIA-0.6mm, F.Cu at (88.2, 94.8)
- added REF**: VIA-0.6mm, Logan:VIA-0.6mm, F.Cu at (87.2, 94.8)
- added REF**: VIA-0.6mm, Logan:VIA-0.6mm, F.Cu at (86.2, 94.8)
- added REF**: VIA-0.6mm, Logan:VIA-0.6mm, F.Cu at (85.2, 103.8)
- added REF**: VIA-0.6mm, Logan:VIA-0.6mm, F.Cu at (85.2, 94.8)
- added REF**: VIA-0.6mm, Logan:VIA-0.6mm, F.Cu at (84.2, 94.8)
- added REF**: VIA-0.6mm, Logan:VIA-0.6mm, F.Cu at (83.2, 94.8)
- added REF**: VIA-0.6mm, Logan:VIA-0.6mm, F.Cu at (82.2, 94.8)
- added REF**: VIA-0.6mm, Logan:VIA-0.6mm, F.Cu at (81.2, 94.8)
- added REF**: VIA-0.6mm, Logan:VIA-0.6mm, F.Cu at (80.2, 94.8)
- added REF**: VIA-0.6mm, Logan:VIA-0.6mm, F.Cu at (79.2, 94.8)
- added REF**: VIA-0.6mm, Logan:VIA-0.6mm, F.Cu at (78.2, 94.8)
- added REF**: VIA-0.6mm, Logan:VIA-0.6mm, F.Cu at (77.2, 94.8)
- added REF**: VIA-0.6mm, Logan:VIA-0.6mm, F.Cu at (76.2, 94.8)
- added REF**: VIA-0.6mm, Logan:VIA-0.6mm, F.Cu at (84.2, 103.8)
- added REF**: VIA-0.6mm, Logan:VIA-0.6mm, F.Cu at (115.2, 93.8)
- added REF**: VIA-0.6mm, Logan:VIA-0.6mm, F.Cu at (114.2, 93.8)
- added REF**: VIA-0.6mm, Logan:VIA-0.6mm, F.Cu at (100.2, 93.8)
- added REF**: VIA-0.6mm, Logan:VIA-0.6mm, F.Cu at (99.2, 93.8)
- added REF**: VIA-0.6mm, Logan:VIA-0.6mm, F.Cu at (98.2, 93.8)
- added REF**: VIA-0.6mm, Logan:VIA-0.6mm, F.Cu at (97.2, 93.8)
- added REF**: VIA-0.6mm, Logan:VIA-0.6mm, F.Cu at (96.2, 93.8)
- added REF**: VIA-0.6mm, Logan:VIA-0.6mm, F.Cu at (95.2, 93.8)
- added REF**: VIA-0.6mm, Logan:VIA-0.6mm, F.Cu at (94.2, 93.8)
- added REF**: VIA-0.6mm, Logan:VIA-0.6mm, F.Cu at (93.2, 93.8)
- added REF**: VIA-0.6mm, Logan:VIA-0.6mm, F.Cu at (83.2, 103.8)
- added REF**: VIA-0.6mm, Logan:VIA-0.6mm, F.Cu at (92.2, 93.8)
- added REF**: VIA-0.6mm, Logan:VIA-0.6mm, F.Cu at (91.2, 93.8)
- added REF**: VIA-0.6mm, Logan:VIA-0.6mm, F.Cu at (90.2, 93.8)
- added REF**: VIA-0.6mm, Logan:VIA-0.6mm, F.Cu at (89.2, 93.8)
- added REF**: VIA-0.6mm, Logan:VIA-0.6mm, F.Cu at (88.2, 93.8)
- added REF**: VIA-0.6mm, Logan:VIA-0.6mm, F.Cu at (87.2, 93.8)
- added REF**: VIA-0.6mm, Logan:VIA-0.6mm, F.Cu at (86.2, 93.8)
- added REF**: VIA-0.6mm, Logan:VIA-0.6mm, F.Cu at (85.2, 93.8)
- added REF**: VIA-0.6mm, Logan:VIA-0.6mm, F.Cu at (84.2, 93.8)
- added REF**: VIA-0.6mm, Logan:VIA-0.6mm, F.Cu at (83.2, 93.8)
- added REF**: VIA-0.6mm, Logan:VIA-0.6mm, F.Cu at (82.2, 103.8)
- added REF**: VIA-0.6mm, Logan:VIA-0.6mm, F.Cu at (82.2, 93.8)
- added REF**: VIA-0.6mm, Logan:VIA-0.6mm, F.Cu at (81.2, 93.8)
- added REF**: VIA-0.6mm, Logan:VIA-0.6mm, F.Cu at (80.2, 93.8)
- added REF**: VIA-0.6mm, Logan:VIA-0.6mm, F.Cu at (79.2, 93.8)
- added REF**: VIA-0.6mm, Logan:VIA-0.6mm, F.Cu at (78.2, 93.8)
- added REF**: VIA-0.6mm, Logan:VIA-0.6mm, F.Cu at (77.2, 93.8)
- added REF**: VIA-0.6mm, Logan:VIA-0.6mm, F.Cu at (76.2, 93.8)
- added REF**: VIA-0.6mm, Logan:VIA-0.6mm, F.Cu at (115.2, 92.8)
- added REF**: VIA-0.6mm, Logan:VIA-0.6mm, F.Cu at (114.2, 92.8)
- added REF**: VIA-0.6mm, Logan:VIA-0.6mm, F.Cu at (100.2, 92.8)
- added REF**: VIA-0.6mm, Logan:VIA-0.6mm, F.Cu at (81.2, 103.8)
- added REF**: VIA-0.6mm, Logan:VIA-0.6mm, F.Cu at (99.2, 92.8)
- added REF**: VIA-0.6mm, Logan:VIA-0.6mm, F.Cu at (98.2, 92.8)
- added REF**: VIA-0.6mm, Logan:VIA-0.6mm, F.Cu at (97.2, 92.8)
- added REF**: VIA-0.6mm, Logan:VIA-0.6mm, F.Cu at (96.2, 92.8)
- added REF**: VIA-0.6mm, Logan:VIA-0.6mm, F.Cu at (95.2, 92.8)
- added REF**: VIA-0.6mm, Logan:VIA-0.6mm, F.Cu at (94.2, 92.8)
- added REF**: VIA-0.6mm, Logan:VIA-0.6mm, F.Cu at (93.2, 92.8)
- added REF**: VIA-0.6mm, Logan:VIA-0.6mm, F.Cu at (92.2, 92.8)
- added REF**: VIA-0.6mm, Logan:VIA-0.6mm, F.Cu at (91.2, 92.8)
- added REF**: VIA-0.6mm, Logan:VIA-0.6mm, F.Cu at (90.2, 92.8)
- added REF**: VIA-0.6mm, Logan:VIA-0.6mm, F.Cu at (80.2, 103.8)
- added REF**: VIA-0.6mm, Logan:VIA-0.6mm, F.Cu at (89.2, 92.8)
- added REF**: VIA-0.6mm, Logan:VIA-0.6mm, F.Cu at (88.2, 92.8)
- added REF**: VIA-0.6mm, Logan:VIA-0.6mm, F.Cu at (87.2, 92.8)
- added REF**: VIA-0.6mm, Logan:VIA-0.6mm, F.Cu at (86.2, 92.8)
- added REF**: VIA-0.6mm, Logan:VIA-0.6mm, F.Cu at (85.2, 92.8)
- added REF**: VIA-0.6mm, Logan:VIA-0.6mm, F.Cu at (84.2, 92.8)
- added REF**: VIA-0.6mm, Logan:VIA-0.6mm, F.Cu at (83.2, 92.8)
- added REF**: VIA-0.6mm, Logan:VIA-0.6mm, F.Cu at (82.2, 92.8)
- added REF**: VIA-0.6mm, Logan:VIA-0.6mm, F.Cu at (81.2, 92.8)
- added REF**: VIA-0.6mm, Logan:VIA-0.6mm, F.Cu at (80.2, 92.8)
- added REF**: VIA-0.6mm, Logan:VIA-0.6mm, F.Cu at (79.2, 103.8)
- added REF**: VIA-0.6mm, Logan:VIA-0.6mm, F.Cu at (79.2, 92.8)
- added REF**: VIA-0.6mm, Logan:VIA-0.6mm, F.Cu at (78.2, 92.8)
- added REF**: VIA-0.6mm, Logan:VIA-0.6mm, F.Cu at (115.2, 91.8)
- added REF**: VIA-0.6mm, Logan:VIA-0.6mm, F.Cu at (114.2, 91.8)
- added REF**: VIA-0.6mm, Logan:VIA-0.6mm, F.Cu at (100.2, 91.8)
- added REF**: VIA-0.6mm, Logan:VIA-0.6mm, F.Cu at (99.2, 91.8)
- added REF**: VIA-0.6mm, Logan:VIA-0.6mm, F.Cu at (98.2, 91.8)
- added REF**: VIA-0.6mm, Logan:VIA-0.6mm, F.Cu at (97.2, 91.8)
- added REF**: VIA-0.6mm, Logan:VIA-0.6mm, F.Cu at (96.2, 91.8)
- added REF**: VIA-0.6mm, Logan:VIA-0.6mm, F.Cu at (95.2, 91.8)
- added REF**: VIA-0.6mm, Logan:VIA-0.6mm, F.Cu at (78.2, 103.8)
- added REF**: VIA-0.6mm, Logan:VIA-0.6mm, F.Cu at (94.2, 91.8)
- added REF**: VIA-0.6mm, Logan:VIA-0.6mm, F.Cu at (93.2, 91.8)
- added REF**: VIA-0.6mm, Logan:VIA-0.6mm, F.Cu at (92.2, 91.8)
- added REF**: VIA-0.6mm, Logan:VIA-0.6mm, F.Cu at (91.2, 91.8)
- added REF**: VIA-0.6mm, Logan:VIA-0.6mm, F.Cu at (90.2, 91.8)
- added REF**: VIA-0.6mm, Logan:VIA-0.6mm, F.Cu at (89.2, 91.8)
- added REF**: VIA-0.6mm, Logan:VIA-0.6mm, F.Cu at (88.2, 91.8)
- added REF**: VIA-0.6mm, Logan:VIA-0.6mm, F.Cu at (87.2, 91.8)
- added REF**: VIA-0.6mm, Logan:VIA-0.6mm, F.Cu at (86.2, 91.8)
- added REF**: VIA-0.6mm, Logan:VIA-0.6mm, F.Cu at (85.2, 91.8)
- added REF**: VIA-0.6mm, Logan:VIA-0.6mm, F.Cu at (77.2, 103.8)
- added REF**: VIA-0.6mm, Logan:VIA-0.6mm, F.Cu at (84.2, 91.8)
- added REF**: VIA-0.6mm, Logan:VIA-0.6mm, F.Cu at (83.2, 91.8)
- added REF**: VIA-0.6mm, Logan:VIA-0.6mm, F.Cu at (82.2, 91.8)
- added REF**: VIA-0.6mm, Logan:VIA-0.6mm, F.Cu at (81.2, 91.8)
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Connections:
- U2 pad 46: Net-(U2-Pad46) -> A
- U2 pad 47: Net-(U2-Pad47) -> B
- U2 pad 48: Net-(U2-Pad48) -> ENC_SW
Routing:
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